File: cad/pcb/saba-fernbedienung/rev1-a/2-steckverbinder.sch (KiCad schematic (older format))
At the start: 12 parts, among them J301 Conn_01x04, J302 Conn_01x04, J303 Conn_01x04, J304 Conn_01x02, J305 Conn_01x04, J306 Conn_01x04, J307 USB_C_Receptacle_USB2.0

Commit message: Add: Steuerschaltung, Codec, Audio
Parts:
- removed D302: SMAJ5.0A, symbol Device:D_TVS
- added C301, C304: 100n, Capacitor_SMD:C_0603_1608Metric, symbol Device:C
- added C302: 10u, Capacitor_SMD:C_1206_3216Metric, symbol Device:C
- added D301: D_TVS_x2_D5V0L2B3W, symbol Device:D_TVS_x2_AAC
- added D303: SMAJ5.0A, Diode_SMD:D_SMA, symbol Diode:SM6T6V8A
- added J303: Micro_SD_Card, symbol Connector:Micro_SD_Card
- added J305: AudioJack3_Ground, symbol Connector:AudioJack3_Ground
- added J308, J309, J310: Conn_01x01, symbol Connector_Generic:Conn_01x01
- added R301, R302: 1k, Resistor_SMD:R_0603_1608Metric, symbol Device:R
- added R303: 0, Resistor_SMD:R_0603_1608Metric, symbol Device:R
- added R304, R308: 1M, Resistor_SMD:R_0603_1608Metric, symbol Device:R
- added R305: 100, Resistor_SMD:R_0603_1608Metric, symbol Device:R
- added U301: TSOP31238, OptoDevice:Vishay_CAST-3Pin, symbol Interface_Optical:TSOP312xx
- C303: renamed from C301; value C -> 100n; Placement No Place -> NP
- D302: renamed from D301; Placement No Place -> NP
- J312: renamed from J307; Placement No Place -> NP
- R306: renamed from R301; Placement No Place -> NP
- R307: renamed from R302; Placement No Place -> NP
- renumbered J303 to J304, J304 to J306, J305 to J307, J306 to J311
Connections:
- net labels added: +3.3V, Audio_Links, Audio_Rechts, Earth, IR_RX, SPI_CS_SDCARD, SPI_MISO, SPI_MOSI, SPI_SCK
- net labels removed: GNDA
- wire segments 53 -> 109
- no-connect marks 4 -> 6
Other:
- note added: "Anschlussstecker Radio Audio"
- note added: "Infrarot Fernbedienung (optional)\n\n"
- note added: "Micro SD Karte (Optional)"
- note added: "Optional: Stereo - 2x 0R"

Commit message: Fix: Div. DRC
Parts:
- added J312: Conn_01x08, symbol Connector_Generic:Conn_01x08
- renumbered J312 to J313
Connections:
- net +5V: now also J312.6 (Pin_6)
- net GND: now also J312.7 (Pin_7)
- net SPI_MOSI: now also J312.3 (Pin_3)
- net SPI_SCK: now also J312.2 (Pin_2)
- net SABA_Reserve: now reaches J311.1 (Pin_1)
- new net LCD_A0: J312.4 (Pin_4)
- new net LCD_BL: J312.5 (Pin_5)
- new net SPI_CS_LCD: J312.1 (Pin_1)
- new net ~RESET: J312.8 (Pin_8)
- no-connect marks 6 -> 11
Other:
- note added: "Infrarot Fernbedienung (optional)"
- note added: "Spannungsversorgung USB (optional)"
- note added: "TFT (optional)"
- note removed: "Infrarot Fernbedienung (optional)\n\n"
- note removed: "Spannungsversorgung USB (optional)\n\n"
- moved on the sheet: C304, R305, U301
Changed lines of the file:
@@
 	1950 3050 1850 3050
 Connection ~ 1950 3000
-NoConn ~ 1850 3200
 NoConn ~ 1850 3300
 NoConn ~ 1850 3400
@@
 Anschlussstecker Radio
 $Comp
-L Connector:USB_C_Receptacle_USB2.0 J312
+L Connector:USB_C_Receptacle_USB2.0 J313
 U 1 1 6005055F
 P 1850 5250
-F 0 "J312" H 1957 6207 50  0000 C CNN
+F 0 "J313" H 1957 6207 50  0000 C CNN
 F 1 "USB_C_Receptacle_USB2.0" H 1957 6116 50  0000 C CNN
 F 2 "" H 2000 5250 50  0001 C CNN
@@
 Wire Notes Line
 	1000 7050 1000 4150
-Text Notes 1050 4200 0    79   ~ 0
-Spannungsversorgung USB (optional)\n\n
-$Comp
-L power:GND #PWR0317
+Text Notes 1050 4100 0    79   ~ 0
+Spannungsversorgung USB (optional)
+$Comp
+L power:GND #PWR0319
 U 1 1 60063A29
 P 1850 6700
-F 0 "#PWR0317" H 1850 6450 50  0001 C CNN
+F 0 "#PWR0319" H 1850 6450 50  0001 C CNN
 F 1 "GND" H 1855 6527 50  0000 C CNN
 F 2 "" H 1850 6700 50  0001 C CNN
@@
 	2450 4950 2700 4950
 $Comp
-L power:GND #PWR0313
+L power:GND #PWR0315
 U 1 1 6006013B
 P 3150 5550
-F 0 "#PWR0313" H 3150 5300 50  0001 C CNN
+F 0 "#PWR0315" H 3150 5300 50  0001 C CNN
 F 1 "GND" H 3155 5377 50  0000 C CNN
 F 2 "" H 3150 5550 50  0001 C CNN
@@
 $EndComp
 $Comp
-L power:GND #PWR0312
+L power:GND #PWR0314
 U 1 1 6005FCD0
 P 2700 5550
-F 0 "#PWR0312" H 2700 5300 50  0001 C CNN
+F 0 "#PWR0314" H 2700 5300 50  0001 C CNN
 F 1 "GND" H 2705 5377 50  0000 C CNN
 F 2 "" H 2700 5550 50  0001 C CNN
@@
 	2450 4650 3550 4650
 $Comp
-L power:GND #PWR0314
+L power:GND #PWR0316
 U 1 1 600712E7
 P 3550 5550
-F 0 "#PWR0314" H 3550 5300 50  0001 C CNN
+F 0 "#PWR0316" H 3550 5300 50  0001 C CNN
 F 1 "GND" H 3555 5377 50  0000 C CNN
 F 2 "" H 3550 5550 50  0001 C CNN
@@
 $EndComp
 $Comp
-L power:GND #PWR0315
+L power:GND #PWR0317
 U 1 1 6007D5DC
 P 4100 5550
-F 0 "#PWR0315" H 4100 5300 50  0001 C CNN
+F 0 "#PWR0317" H 4100 5300 50  0001 C CNN
 F 1 "GND" H 4105 5377 50  0000 C CNN
 F 2 "" H 4100 5550 50  0001 C CNN
@@
 L Interface_Optical:TSOP312xx U301
 U 1 1 60019665
-P 6650 4850
-F 0 "U301" H 6638 5275 50  0000 C CNN
-F 1 "TSOP31238" H 6638 5184 50  0000 C CNN
-F 2 "OptoDevice:Vishay_CAST-3Pin" H 6600 4475 50  0001 C CNN
-F 3 "http://www.vishay.com/docs/82492/tsop312.pdf" H 7300 5150 50  0001 C CNN
-	1    6650 4850
-	1    0    0    -1
-$EndComp
-$Comp
-L power:GND #PWR0311
+P 8050 4850
+F 0 "U301" H 8038 5275 50  0000 C CNN
+F 1 "TSOP31238" H 8038 5184 50  0000 C CNN
+F 2 "OptoDevice:Vishay_CAST-3Pin" H 8000 4475 50  0001 C CNN
+F 3 "http://www.vishay.com/docs/82492/tsop312.pdf" H 8700 5150 50  0001 C CNN
+	1    8050 4850
+	1    0    0    -1
+$EndComp
+$Comp
+L power:GND #PWR0312
 U 1 1 6001F94B
-P 7150 5200
-F 0 "#PWR0311" H 7150 4950 50  0001 C CNN
-F 1 "GND" H 7155 5027 50  0000 C CNN
-F 2 "" H 7150 5200 50  0001 C CNN
-F 3 "" H 7150 5200 50  0001 C CNN
-	1    7150 5200
-	1    0    0    -1
-$EndComp
-Text GLabel 7300 4850 2    50   Output ~ 0
+P 8550 5200
+F 0 "#PWR0312" H 8550 4950 50  0001 C CNN
+F 1 "GND" H 8555 5027 50  0000 C CNN
+F 2 "" H 8550 5200 50  0001 C CNN
+F 3 "" H 8550 5200 50  0001 C CNN
+	1    8550 5200
+	1    0    0    -1
+$EndComp
+Text GLabel 8700 4850 2    50   Output ~ 0
 IR_RX
 Wire Wire Line
-	7050 4850 7300 4850
-Wire Wire Line
-	7050 5050 7150 5050
-Wire Wire Line
-	7150 5050 7150 5200
-Wire Notes Line
-	6000 4150 9200 4150
-Wire Notes Line
-	9200 4150 9200 5900
-Wire Notes Line
-	9200 5900 6000 5900
-Wire Notes Line
-	6000 5900 6000 4150
-Text Notes 6050 4200 0    79   ~ 0
-Infrarot Fernbedienung (optional)\n\n
+	8450 4850 8700 4850
+Wire Wire Line
+	8450 5050 8550 5050
+Wire Wire Line
+	8550 5050 8550 5200
+Wire Notes Line
+	7400 4150 10600 4150
+Wire Notes Line
+	10600 4150 10600 5900
+Wire Notes Line
+	10600 5900 7400 5900
+Wire Notes Line
+	7400 5900 7400 4150
+Text Notes 7450 4100 0    79   ~ 0
+Infrarot Fernbedienung (optional)
 $Comp
 L Connector:AudioJack3_Ground J305
@@
 Connection ~ 4450 2350
 Wire Wire Line
-	7800 4650 7050 4650
-Wire Wire Line
-	7800 4750 7800 4650
-Wire Wire Line
-	7800 5150 7800 5050
-Connection ~ 7800 4650
-Wire Wire Line
-	8100 4650 7800 4650
-Wire Wire Line
-	8500 4650 8400 4650
-Wire Wire Line
-	8500 4550 8500 4650
+	9200 4650 8450 4650
+Wire Wire Line
+	9200 4750 9200 4650
+Wire Wire Line
+	9200 5150 9200 5050
+Connection ~ 9200 4650
+Wire Wire Line
+	9500 4650 9200 4650
+Wire Wire Line
+	9900 4650 9800 4650
+Wire Wire Line
+	9900 4550 9900 4650
 $Comp
 L power:+3.3V #PWR0308
 U 1 1 60021397
-P 8500 4550
-F 0 "#PWR0308" H 8500 4400 50  0001 C CNN
-F 1 "+3.3V" H 8515 4723 50  0000 C CNN
-F 2 "" H 8500 4550 50  0001 C CNN
-F 3 "" H 8500 4550 50  0001 C CNN
-	1    8500 4550
-	1    0    0    -1
-$EndComp
-$Comp
-L power:GND #PWR0310
+P 9900 4550
+F 0 "#PWR0308" H 9900 4400 50  0001 C CNN
+F 1 "+3.3V" H 9915 4723 50  0000 C CNN
+F 2 "" H 9900 4550 50  0001 C CNN
+F 3 "" H 9900 4550 50  0001 C CNN
+	1    9900 4550
+	1    0    0    -1
+$EndComp
+$Comp
+L power:GND #PWR0311
 U 1 1 60020161
-P 7800 5150
-F 0 "#PWR0310" H 7800 4900 50  0001 C CNN
-F 1 "GND" H 7805 4977 50  0000 C CNN
-F 2 "" H 7800 5150 50  0001 C CNN
-F 3 "" H 7800 5150 50  0001 C CNN
-	1    7800 5150
+P 9200 5150
+F 0 "#PWR0311" H 9200 4900 50  0001 C CNN
+F 1 "GND" H 9205 4977 50  0000 C CNN
+F 2 "" H 9200 5150 50  0001 C CNN
+F 3 "" H 9200 5150 50  0001 C CNN
+	1    9200 5150
 	1    0    0    -1
 $EndComp
@@
 L Device:C C304
 U 1 1 6001EC41
-P 7800 4900
-F 0 "C304" H 7915 4991 50  0000 L CNN
-F 1 "100n" H 7915 4900 50  0000 L CNN
-F 2 "Capacitor_SMD:C_0603_1608Metric" H 7838 4750 50  0001 C CNN
-F 3 "~" H 7800 4900 50  0001 C CNN
-F 4 "" H 7915 4809 50  0000 L CNN "Placement"
-	1    7800 4900
+P 9200 4900
+F 0 "C304" H 9315 4991 50  0000 L CNN
+F 1 "100n" H 9315 4900 50  0000 L CNN
+F 2 "Capacitor_SMD:C_0603_1608Metric" H 9238 4750 50  0001 C CNN
+F 3 "~" H 9200 4900 50  0001 C CNN
+F 4 "" H 9315 4809 50  0000 L CNN "Placement"
+	1    9200 4900
 	1    0    0    -1
 $EndComp
@@
 L Device:R R?
 U 1 1 6001BDE1
-P 8250 4650
+P 9650 4650
 AR Path="/5FFC49DA/6001BDE1" Ref="R?"  Part="1"
 AR Path="/6002EA57/6001BDE1" Ref="R305"  Part="1"
-F 0 "R305" H 8180 4559 50  0000 R CNN
-F 1 "100" H 8180 4650 50  0000 R CNN
-F 2 "Resistor_SMD:R_0603_1608Metric" V 8180 4650 50  0001 C CNN
-F 3 "~" H 8250 4650 50  0001 C CNN
-F 4 "" V 8250 4700 50  0000 R CNN "Placement"
-	1    8250 4650
+F 0 "R305" H 9580 4559 50  0000 R CNN
+F 1 "100" H 9580 4650 50  0000 R CNN
+F 2 "Resistor_SMD:R_0603_1608Metric" V 9580 4650 50  0001 C CNN
+F 3 "~" H 9650 4650 50  0001 C CNN
+F 4 "" V 9650 4700 50  0000 R CNN "Placement"
+	1    9650 4650
 	0    -1   -1   0
 $EndComp
@@
 $EndComp
 $Comp
-L power:Earth #PWR0316
+L power:Earth #PWR0318
 U 1 1 600AE860
 P 1550 6700
-F 0 "#PWR0316" H 1550 6450 50  0001 C CNN
+F 0 "#PWR0318" H 1550 6450 50  0001 C CNN
 F 1 "Earth" H 1550 6550 50  0001 C CNN
 F 2 "" H 1550 6700 50  0001 C CNN
@@
 	4450 3100 4450 2600
 Connection ~ 4450 2600
+Text GLabel 2250 3200 2    50   Output ~ 0
+SABA_Reserve
+Wire Wire Line
+	2250 3200 1850 3200
+$Comp
+L Connector_Generic:Conn_01x08 J312
+U 1 1 60A4DF30
+P 6600 4900
+F 0 "J312" H 6680 4937 50  0000 L CNN
+F 1 "Conn_01x08" H 6680 4846 50  0000 L CNN
+F 2 "" H 6600 4900 50  0001 C CNN
+F 3 "~" H 6600 4900 50  0001 C CNN
+F 4 "NP" H 6680 4755 50  0000 L CNN "Placement"
+	1    6600 4900
+	1    0    0    -1
+$EndComp
+Text GLabel 6150 4600 0    50   Input ~ 0
+SPI_CS_LCD
+Text GLabel 6150 4700 0    50   Input ~ 0
+SPI_SCK
+Text GLabel 6150 4800 0    50   Input ~ 0
+SPI_MOSI
+Text GLabel 6150 5300 0    50   Input ~ 0
+~RESET
+Text GLabel 6150 4900 0    50   Input ~ 0
+LCD_A0
+Text GLabel 6150 5000 0    50   Input ~ 0
+LCD_BL
+$Comp
+L power:+5V #PWR0310
+U 1 1 60A526F1
+P 5650 5050
+F 0 "#PWR0310" H 5650 4900 50  0001 C CNN
+F 1 "+5V" H 5665 5223 50  0000 C CNN
+F 2 "" H 5650 5050 50  0001 C CNN
+F 3 "" H 5650 5050 50  0001 C CNN
+	1    5650 5050
+	1    0    0    -1
+$EndComp
+$Comp
+L power:GND #PWR0313
+U 1 1 60A52FFC
+P 5650 5250
+F 0 "#PWR0313" H 5650 5000 50  0001 C CNN
+F 1 "GND" H 5655 5077 50  0000 C CNN
+F 2 "" H 5650 5250 50  0001 C CNN
+F 3 "" H 5650 5250 50  0001 C CNN
+	1    5650 5250
+	1    0    0    -1
+$EndComp
+Wire Wire Line
+	6150 4600 6400 4600
+Wire Wire Line
+	6150 4700 6400 4700
+Wire Wire Line
+	6150 4800 6400 4800
+Wire Wire Line
+	6150 4900 6400 4900
+Wire Wire Line
+	6400 5000 6150 5000
+Wire Wire Line
+	6400 5100 5650 5100
+Wire Wire Line
+	5650 5100 5650 5050
+Wire Wire Line
+	6400 5200 5650 5200
+Wire Wire Line
+	5650 5200 5650 5250
+Wire Wire Line
+	6400 5300 6150 5300
+Text Notes 5550 4100 0    79   ~ 0
+TFT (optional)
+Wire Notes Line
+	5500 4150 7250 4150
+Wire Notes Line
+	7250 4150 7250 5900
+Wire Notes Line
+	7250 5900 5500 5900
+Wire Notes Line
+	5500 5900 5500 4150
+NoConn ~ 2450 5150
+NoConn ~ 2450 5250
+NoConn ~ 2450 5350
+NoConn ~ 2450 5450
+NoConn ~ 2450 5750
+NoConn ~ 2450 5850
 $EndSCHEMATC

Commit message: New: Bauteil - Pad Zuordnungen
Parts:
- removed J305: AudioJack3_Ground, symbol Connector:AudioJack3_Ground
- added J305: AudioJack3, Connector_Audio:Jack_3.5mm_CUI_SJ-3523-SMT_Horizontal, symbol Connector:AudioJack3
- D301: footprint (none) -> Package_TO_SOT_SMD:SOT-323_SC-70
- J301, J302, J304, J307, J311: footprint (none) -> Connector_PinHeader_2.54mm:PinHeader_1x04_P2.54mm_Vertical
- J303: footprint (none) -> Connector_Card:microSD_HC_Hirose_DM3AT-SF-PEJM5
- J306: footprint (none) -> Connector_PinHeader_2.54mm:PinHeader_1x02_P2.54mm_Vertical
- J308, J309, J310: footprint (none) -> Connector_PinHeader_2.54mm:PinHeader_1x01_P2.54mm_Vertical
- J312: footprint (none) -> Connector_PinHeader_2.54mm:PinHeader_2x04_P2.54mm_Vertical
- J313: footprint (none) -> Connector_USB:USB_C_Receptacle_HRO_TYPE-C-31-M-12
Connections:
- net Earth: now also J305.T
- net at D301.2 (A2), J310.1 (Pin_1), R303.1: now also J305.R
- net at D301.1 (A1), J309.1 (Pin_1), R301.2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: now also J305.S
Changed lines of the file:
@@
 F 0 "J306" H 2000 2500 50  0000 C CNN
 F 1 "Conn_01x02" H 2000 2400 50  0000 C CNN
-F 2 "" H 1650 2500 50  0001 C CNN
+F 2 "Connector_PinHeader_2.54mm:PinHeader_1x02_P2.54mm_Vertical" H 1650 2500 50  0001 C CNN
 F 3 "~" H 1650 2500 50  0001 C CNN
 	1    1650 2500
@@
 F 0 "J301" H 2000 1300 50  0000 C CNN
 F 1 "Conn_01x04" H 2000 1200 50  0000 C CNN
-F 2 "" H 1650 1250 50  0001 C CNN
+F 2 "Connector_PinHeader_2.54mm:PinHeader_1x04_P2.54mm_Vertical" H 1650 1250 50  0001 C CNN
 F 3 "~" H 1650 1250 50  0001 C CNN
 	1    1650 1250
@@
 F 0 "J302" H 2000 1750 50  0000 C CNN
 F 1 "Conn_01x04" H 2000 1650 50  0000 C CNN
-F 2 "" H 1650 1700 50  0001 C CNN
+F 2 "Connector_PinHeader_2.54mm:PinHeader_1x04_P2.54mm_Vertical" H 1650 1700 50  0001 C CNN
 F 3 "~" H 1650 1700 50  0001 C CNN
 	1    1650 1700
@@
 F 0 "J304" H 2000 2150 50  0000 C CNN
 F 1 "Conn_01x04" H 2000 2050 50  0000 C CNN
-F 2 "" H 1650 2150 50  0001 C CNN
+F 2 "Connector_PinHeader_2.54mm:PinHeader_1x04_P2.54mm_Vertical" H 1650 2150 50  0001 C CNN
 F 3 "~" H 1650 2150 50  0001 C CNN
 	1    1650 2150
@@
 F 0 "J307" H 2000 2850 50  0000 C CNN
 F 1 "Conn_01x04" H 2000 2750 50  0000 C CNN
-F 2 "" H 1650 2850 50  0001 C CNN
+F 2 "Connector_PinHeader_2.54mm:PinHeader_1x04_P2.54mm_Vertical" H 1650 2850 50  0001 C CNN
 F 3 "~" H 1650 2850 50  0001 C CNN
 	1    1650 2850
@@
 F 0 "J311" H 2000 3300 50  0000 C CNN
 F 1 "Conn_01x04" H 2000 3200 50  0000 C CNN
-F 2 "" H 1650 3300 50  0001 C CNN
+F 2 "Connector_PinHeader_2.54mm:PinHeader_1x04_P2.54mm_Vertical" H 1650 3300 50  0001 C CNN
 F 3 "~" H 1650 3300 50  0001 C CNN
 	1    1650 3300
@@
 F 0 "J313" H 1957 6207 50  0000 C CNN
 F 1 "USB_C_Receptacle_USB2.0" H 1957 6116 50  0000 C CNN
-F 2 "" H 2000 5250 50  0001 C CNN
+F 2 "Connector_USB:USB_C_Receptacle_HRO_TYPE-C-31-M-12" H 2000 5250 50  0001 C CNN
 F 3 "https://www.usb.org/sites/default/files/documents/usb_type-c.zip" H 2000 5250 50  0001 C CNN
 F 4 "NP" H 1957 6025 50  0000 C CNN "Placement"
@@
 F 0 "J303" H 7450 2817 50  0000 C CNN
 F 1 "Micro_SD_Card" H 7450 2726 50  0000 C CNN
-F 2 "" H 8650 2400 50  0001 C CNN
+F 2 "Connector_Card:microSD_HC_Hirose_DM3AT-SF-PEJM5" H 8650 2400 50  0001 C CNN
 F 3 "http://katalog.we-online.de/em/datasheet/693072010801.pdf" H 7500 2100 50  0001 C CNN
 	1    7500 2100
@@
 Text Notes 7450 4100 0    79   ~ 0
 Infrarot Fernbedienung (optional)
-$Comp
-L Connector:AudioJack3_Ground J305
-U 1 1 6003F711
-P 4150 2250
-F 0 "J305" H 4132 2575 50  0000 C CNN
-F 1 "AudioJack3_Ground" H 4132 2484 50  0000 C CNN
-F 2 "" H 4150 2250 50  0001 C CNN
-F 3 "~" H 4150 2250 50  0001 C CNN
-	1    4150 2250
-	1    0    0    -1
-$EndComp
-Wire Wire Line
-	4150 2550 4150 2600
 Wire Wire Line
 	4350 2350 4450 2350
 Wire Wire Line
 	4450 2350 4450 2600
-Wire Wire Line
-	4450 2600 4150 2600
-Connection ~ 4150 2600
-Wire Wire Line
-	4150 2600 4150 2650
 Text GLabel 6000 1550 1    50   Input ~ 0
 Audio_Links
@@
 F 0 "J308" H 5350 2850 50  0000 L CNN
 F 1 "Conn_01x01" H 5600 2850 50  0000 L CNN
-F 2 "" H 5250 2850 50  0001 C CNN
+F 2 "Connector_PinHeader_2.54mm:PinHeader_1x01_P2.54mm_Vertical" H 5250 2850 50  0001 C CNN
 F 3 "~" H 5250 2850 50  0001 C CNN
 	1    5250 2850
@@
 F 0 "J309" H 5500 2850 50  0000 L CNN
 F 1 "Conn_01x01" H 5750 2850 50  0000 L CNN
-F 2 "" H 5400 2850 50  0001 C CNN
+F 2 "Connector_PinHeader_2.54mm:PinHeader_1x01_P2.54mm_Vertical" H 5400 2850 50  0001 C CNN
 F 3 "~" H 5400 2850 50  0001 C CNN
 	1    5400 2850
@@
 F 0 "J310" H 5650 2850 50  0000 L CNN
 F 1 "Conn_01x01" H 5900 2850 50  0000 L CNN
-F 2 "" H 5550 2850 50  0001 C CNN
+F 2 "Connector_PinHeader_2.54mm:PinHeader_1x01_P2.54mm_Vertical" H 5550 2850 50  0001 C CNN
 F 3 "~" H 5550 2850 50  0001 C CNN
 	1    5550 2850
@@
 $EndComp
 $Comp
-L power:Earth #PWR0306
-U 1 1 600ACF99
-P 4150 2650
-F 0 "#PWR0306" H 4150 2400 50  0001 C CNN
-F 1 "Earth" H 4150 2500 50  0001 C CNN
-F 2 "" H 4150 2650 50  0001 C CNN
-F 3 "~" H 4150 2650 50  0001 C CNN
-	1    4150 2650
-	1    0    0    -1
-$EndComp
-$Comp
 L power:Earth #PWR0307
 U 1 1 600ADE98
@@
 F 0 "D301" V 4554 3180 50  0000 L CNN
 F 1 "D_TVS_x2_D5V0L2B3W" V 4750 2200 50  0000 L CNN
-F 2 "" H 4450 3100 50  0001 C CNN
+F 2 "Package_TO_SOT_SMD:SOT-323_SC-70" H 4450 3100 50  0001 C CNN
 F 3 "https://www.diodes.com/assets/Datasheets/D5V0L2B3W.pdf" H 4450 3100 50  0001 C CNN
 	1    4600 3100
@@
 F 0 "J312" H 6680 4937 50  0000 L CNN
 F 1 "Conn_01x08" H 6680 4846 50  0000 L CNN
-F 2 "" H 6600 4900 50  0001 C CNN
+F 2 "Connector_PinHeader_2.54mm:PinHeader_2x04_P2.54mm_Vertical" H 6600 4900 50  0001 C CNN
 F 3 "~" H 6600 4900 50  0001 C CNN
 F 4 "NP" H 6680 4755 50  0000 L CNN "Placement"
@@
 NoConn ~ 2450 5750
 NoConn ~ 2450 5850
+$Comp
+L power:Earth #PWR0306
+U 1 1 600ACF99
+P 4350 2650
+F 0 "#PWR0306" H 4350 2400 50  0001 C CNN
+F 1 "Earth" H 4350 2500 50  0001 C CNN
+F 2 "" H 4350 2650 50  0001 C CNN
+F 3 "~" H 4350 2650 50  0001 C CNN
+	1    4350 2650
+	1    0    0    -1
+$EndComp
+Wire Wire Line
+	4350 2600 4350 2650
+Wire Wire Line
+	4450 2600 4350 2600
+$Comp
+L Connector:AudioJack3 J305
+U 1 1 60BB0BE0
+P 4150 2250
+F 0 "J305" H 4132 2575 50  0000 C CNN
+F 1 "AudioJack3" H 4132 2484 50  0000 C CNN
+F 2 "Connector_Audio:Jack_3.5mm_CUI_SJ-3523-SMT_Horizontal" H 4150 2250 50  0001 C CNN
+F 3 "~" H 4150 2250 50  0001 C CNN
+	1    4150 2250
+	1    0    0    -1
+$EndComp
 $EndSCHEMATC

Commit message: Add: Bauteiltypen Digikey...
viele Bauteile von WE da hoffentlich lange gueltig...
Parts:
- C301, C303, C304: Bauteil (none) -> WE 885382206004
- C302: Bauteil (none) -> WE 885012208069
- D301: value D_TVS_x2_D5V0L2B3W -> 5V; Bauteil (none) -> Diodes D5V0L2B3W
- D302: Bauteil (none) -> Vishay B140-E3/61T
- D303: Bauteil (none) -> SMAJ5.0A-13-F
- J303: Bauteil (none) -> Hirose DM3AT-SF-PEJM5
- J305: Bauteil (none) -> CUI SJ-3523-SMT-TR
- J313: Bauteil (none) -> GCT USB4125-GF-A
- U301: Bauteil (none) -> Vishay TSOP31238
Changed lines of the file:
@@
 F 3 "https://www.usb.org/sites/default/files/documents/usb_type-c.zip" H 2000 5250 50  0001 C CNN
 F 4 "NP" H 1957 6025 50  0000 C CNN "Placement"
+F 5 "GCT USB4125-GF-A" H 1850 5250 50  0001 C CNN "Bauteil"
 	1    1850 5250
 	1    0    0    -1
@@
 F 3 "~" H 3550 4900 50  0001 C CNN
 F 4 "NP" H 3665 4809 50  0000 L CNN "Placement"
+F 5 "WE 885382206004" H 3550 4900 50  0001 C CNN "Bauteil"
 	1    3550 4900
 	1    0    0    -1
@@
 F 3 "http://www.vishay.com/docs/88946/b120.pdf" H 4650 4650 50  0001 C CNN
 F 4 "NP" H 4650 4525 50  0000 C CNN "Placement"
+F 5 "Vishay B140-E3/61T" H 4650 4650 50  0001 C CNN "Bauteil"
 	1    4650 4650
 	-1   0    0    1
@@
 F 2 "Connector_Card:microSD_HC_Hirose_DM3AT-SF-PEJM5" H 8650 2400 50  0001 C CNN
 F 3 "http://katalog.we-online.de/em/datasheet/693072010801.pdf" H 7500 2100 50  0001 C CNN
+F 4 "Hirose DM3AT-SF-PEJM5" H 7500 2100 50  0001 C CNN "Bauteil"
 	1    7500 2100
 	-1   0    0    -1
@@
 F 3 "~" H 9650 2350 50  0001 C CNN
 F 4 "" H 9765 2259 50  0000 L CNN "Placement"
+F 5 "WE 885382206004" H 9650 2350 50  0001 C CNN "Bauteil"
 	1    9650 2350
 	1    0    0    -1
@@
 F 3 "~" H 10150 2350 50  0001 C CNN
 F 4 "" H 10265 2259 50  0000 L CNN "Placement"
+F 5 "WE 885012208069" H 10150 2350 50  0001 C CNN "Bauteil"
 	1    10150 2350
 	1    0    0    -1
@@
 F 2 "OptoDevice:Vishay_CAST-3Pin" H 8000 4475 50  0001 C CNN
 F 3 "http://www.vishay.com/docs/82492/tsop312.pdf" H 8700 5150 50  0001 C CNN
+F 4 "Vishay TSOP31238" H 8050 4850 50  0001 C CNN "Bauteil"
 	1    8050 4850
 	1    0    0    -1
@@
 F 3 "~" H 9200 4900 50  0001 C CNN
 F 4 "" H 9315 4809 50  0000 L CNN "Placement"
+F 5 "WE 885382206004" H 9200 4900 50  0001 C CNN "Bauteil"
 	1    9200 4900
 	1    0    0    -1
@@
 F 3 "" H 4050 4900 50  0001 C CNN
 F 4 "NP" V 4191 4980 50  0000 L CNN "Placement"
+F 5 "SMAJ5.0A-13-F" V 4100 4900 50  0001 C CNN "Bauteil"
 	1    4100 4900
 	0    1    1    0
@@
 U 1 1 609A1EE5
 P 4600 3100
-F 0 "D301" V 4554 3180 50  0000 L CNN
-F 1 "D_TVS_x2_D5V0L2B3W" V 4750 2200 50  0000 L CNN
+F 0 "D301" V 4700 2750 50  0000 L CNN
+F 1 "5V" V 4800 2800 50  0000 L CNN
 F 2 "Package_TO_SOT_SMD:SOT-323_SC-70" H 4450 3100 50  0001 C CNN
 F 3 "https://www.diodes.com/assets/Datasheets/D5V0L2B3W.pdf" H 4450 3100 50  0001 C CNN
+F 4 "Diodes D5V0L2B3W" V 4600 3100 50  0001 C CNN "Bauteil"
 	1    4600 3100
 	0    1    1    0
@@
 F 2 "Connector_Audio:Jack_3.5mm_CUI_SJ-3523-SMT_Horizontal" H 4150 2250 50  0001 C CNN
 F 3 "~" H 4150 2250 50  0001 C CNN
+F 4 "CUI SJ-3523-SMT-TR" H 4150 2250 50  0001 C CNN "Bauteil"
 	1    4150 2250
 	1    0    0    -1

Commit message: Sicherung
Connections:
- net SABA_Reserve: no longer names the net of J311.1 (Pin_1)
- no-connect marks 11 -> 12
Changed lines of the file:
@@
 	4450 3100 4450 2600
 Connection ~ 4450 2600
-Text GLabel 2250 3200 2    50   Output ~ 0
-SABA_Reserve
-Wire Wire Line
-	2250 3200 1850 3200
 $Comp
 L Connector_Generic:Conn_01x08 J312
@@
 	1    0    0    -1
 $EndComp
+NoConn ~ 1850 3200
 $EndSCHEMATC

Commit message: Sicherung
Connections:
- net LCD_A0: now also J312.8 (Pin_8); no longer J312.4 (Pin_4)
- net ~RESET: now also J312.4 (Pin_4); no longer J312.8 (Pin_8)
Changed lines of the file:
@@
 Text GLabel 6150 4800 0    50   Input ~ 0
 SPI_MOSI
+Text GLabel 6150 4900 0    50   Input ~ 0
+~RESET
 Text GLabel 6150 5300 0    50   Input ~ 0
-~RESET
-Text GLabel 6150 4900 0    50   Input ~ 0
 LCD_A0
 Text GLabel 6150 5000 0    50   Input ~ 0
