File: cad/pcb/saba-fernbedienung/rev1-a/6-audio.sch (KiCad schematic (older format))
At the start: 52 parts, among them U701 AD8656, U702 VS1053, Y701 12,288MHz

Commit message: Fix: Div. DRC
Parts:
- renumbered C713 to C710, C710 to C711, C711 to C712, C712 to C713
Connections:
- no-connect marks 3 -> 5
Changed lines of the file:
@@
 AR Path="/60135668/604F8AD6" Ref="C?"  Part="1"
 AR Path="/6044FE50/604F8AD6" Ref="C?"  Part="1"
-AR Path="/6041BFCD/604F8AD6" Ref="C712"  Part="1"
-F 0 "C712" H 5865 2341 50  0000 L CNN
+AR Path="/6041BFCD/604F8AD6" Ref="C713"  Part="1"
+F 0 "C713" H 5865 2341 50  0000 L CNN
 F 1 "100n" H 5865 2250 50  0000 L CNN
 F 2 "Capacitor_SMD:C_0603_1608Metric" H 5788 2100 50  0001 C CNN
@@
 AR Path="/60135668/604F8ADD" Ref="C?"  Part="1"
 AR Path="/6044FE50/604F8ADD" Ref="C?"  Part="1"
-AR Path="/6041BFCD/604F8ADD" Ref="C711"  Part="1"
-F 0 "C711" H 5415 2341 50  0000 L CNN
+AR Path="/6041BFCD/604F8ADD" Ref="C712"  Part="1"
+F 0 "C712" H 5415 2341 50  0000 L CNN
 F 1 "100n" H 5415 2250 50  0000 L CNN
 F 2 "Capacitor_SMD:C_0603_1608Metric" H 5338 2100 50  0001 C CNN
@@
 AR Path="/60135668/604F8AE4" Ref="C?"  Part="1"
 AR Path="/6044FE50/604F8AE4" Ref="C?"  Part="1"
-AR Path="/6041BFCD/604F8AE4" Ref="C710"  Part="1"
-F 0 "C710" H 4965 2341 50  0000 L CNN
+AR Path="/6041BFCD/604F8AE4" Ref="C711"  Part="1"
+F 0 "C711" H 4965 2341 50  0000 L CNN
 F 1 "100n" H 4965 2250 50  0000 L CNN
 F 2 "Capacitor_SMD:C_0603_1608Metric" H 4888 2100 50  0001 C CNN
@@
 Wire Wire Line
 	1200 4100 1200 4400
-Text GLabel 1750 2950 0    50   Input ~ 0
+Text GLabel 1750 2950 0    50   Output ~ 0
 SPI_MISO
 Text GLabel 1750 3050 0    50   Input ~ 0
@@
 Text GLabel 1750 3350 0    50   Input ~ 0
 SPI_DCS_VS1053
-Text GLabel 1750 3450 0    50   Input ~ 0
+Text GLabel 1750 3450 0    50   Output ~ 0
 VS1053_DREQ
 Text GLabel 1750 3600 0    50   Input ~ 0
@@
 AR Path="/60135668/607C4A6B" Ref="C?"  Part="1"
 AR Path="/6044FE50/607C4A6B" Ref="C?"  Part="1"
-AR Path="/6041BFCD/607C4A6B" Ref="C713"  Part="1"
-F 0 "C713" H 8565 2291 50  0000 L CNN
+AR Path="/6041BFCD/607C4A6B" Ref="C710"  Part="1"
+F 0 "C710" H 8565 2291 50  0000 L CNN
 F 1 "100n" H 8565 2200 50  0000 L CNN
 F 2 "Capacitor_SMD:C_0603_1608Metric" H 8488 2050 50  0001 C CNN
@@
 	9200 2100 9200 1700
 Connection ~ 9200 1700
-Text GLabel 10650 1700 1    50   Input ~ 0
+Text GLabel 10650 1700 1    50   Output ~ 0
 Audio_Links
 Wire Wire Line
@@
 Text Label 9000 4100 1    50   ~ 0
 rechts
-Text GLabel 10650 3550 1    50   Input ~ 0
+Text GLabel 10650 3550 1    50   Output ~ 0
 Audio_Rechts
 Wire Notes Line
@@
 NoConn ~ 4400 4450
 NoConn ~ 4400 4550
+NoConn ~ 2050 3750
+NoConn ~ 4400 3950
 $EndSCHEMATC

Commit message: New: Bauteil - Pad Zuordnungen
Parts:
- L701: footprint (none) -> local:WE-LQ; Type TDK TCK-154 -> WE 744045004
- R707: value 100k -> 1M
- RV701, RV702: footprint (none) -> Potentiometer_SMD:Potentiometer_Vishay_TS53YL_Vertical
- U701: footprint (none) -> Package_SO:SOIC-8_3.9x4.9mm_P1.27mm
- U702: footprint (none) -> Package_QFP:LQFP-48_7x7mm_P0.5mm
- Y701: footprint (none) -> Crystal:Crystal_SMD_HC49-SD
Changed lines of the file:
@@
 F 0 "U702" H 4050 8600 50  0000 C CNN
 F 1 "VS1053" H 3200 7200 50  0000 C CNN
-F 2 "" H 3150 5450 50  0001 C CNN
+F 2 "Package_QFP:LQFP-48_7x7mm_P0.5mm" H 3150 5450 50  0001 C CNN
 F 3 "" H 3150 5450 50  0001 C CNN
 	1    3150 5450
@@
 F 0 "Y701" V 5254 3231 50  0000 L CNN
 F 1 "12,288MHz" V 5345 3231 50  0000 L CNN
-F 2 "" H 5300 3100 50  0001 C CNN
+F 2 "Crystal:Crystal_SMD_HC49-SD" H 5300 3100 50  0001 C CNN
 F 3 "~" H 5300 3100 50  0001 C CNN
 	1    5300 3100
@@
 AR Path="/6041BFCD/605938CA" Ref="R707"  Part="1"
 F 0 "R707" H 4830 3009 50  0000 R CNN
-F 1 "100k" H 4830 3100 50  0000 R CNN
+F 1 "1M" H 4830 3100 50  0000 R CNN
 F 2 "Resistor_SMD:R_0603_1608Metric" V 4830 3100 50  0001 C CNN
 F 3 "~" H 4900 3100 50  0001 C CNN
@@
 F 0 "U701" H 9700 1433 50  0000 C CNN
 F 1 "AD8656" H 9700 1524 50  0000 C CNN
-F 2 "" H 9700 1800 50  0001 C CNN
+F 2 "Package_SO:SOIC-8_3.9x4.9mm_P1.27mm" H 9700 1800 50  0001 C CNN
 F 3 "https://www.analog.com/media/en/technical-documentation/data-sheets/AD8655_8656.pdf" H 9700 1800 50  0001 C CNN
 	1    9700 1800
@@
 F 0 "U701" H 9700 3283 50  0000 C CNN
 F 1 "AD8656" H 9700 3374 50  0000 C CNN
-F 2 "" H 9700 3650 50  0001 C CNN
+F 2 "Package_SO:SOIC-8_3.9x4.9mm_P1.27mm" H 9700 3650 50  0001 C CNN
 F 3 "https://www.analog.com/media/en/technical-documentation/data-sheets/AD8655_8656.pdf" H 9700 3650 50  0001 C CNN
 	2    9700 3650
@@
 F 0 "U701" H 2108 6796 50  0000 L CNN
 F 1 "AD8656" H 2108 6705 50  0000 L CNN
-F 2 "" H 2150 6750 50  0001 C CNN
+F 2 "Package_SO:SOIC-8_3.9x4.9mm_P1.27mm" H 2150 6750 50  0001 C CNN
 F 3 "https://www.analog.com/media/en/technical-documentation/data-sheets/AD8655_8656.pdf" H 2150 6750 50  0001 C CNN
 	3    2150 6750
@@
 F 0 "L701" V 1290 6400 50  0000 C CNN
 F 1 "4,7u" V 1199 6400 50  0000 C CNN
-F 2 "" H 1100 6400 50  0001 C CNN
+F 2 "local:WE-LQ" H 1100 6400 50  0001 C CNN
 F 3 "~" H 1100 6400 50  0001 C CNN
-F 4 "TDK TCK-154" V 1100 6400 50  0001 C CNN "Type"
+F 4 "WE 744045004" V 1100 6400 50  0001 C CNN "Type"
 	1    1100 6400
 	0    -1   -1   0
@@
 F 0 "RV701" H 9131 1496 50  0000 R CNN
 F 1 "22k lin" H 9131 1405 50  0000 R CNN
-F 2 "" H 9200 1450 50  0001 C CNN
+F 2 "Potentiometer_SMD:Potentiometer_Vishay_TS53YL_Vertical" H 9200 1450 50  0001 C CNN
 F 3 "~" H 9200 1450 50  0001 C CNN
 	1    9200 1450
@@
 F 0 "RV702" H 9131 3346 50  0000 R CNN
 F 1 "22k lin" H 9131 3255 50  0000 R CNN
-F 2 "" H 9200 3300 50  0001 C CNN
+F 2 "Potentiometer_SMD:Potentiometer_Vishay_TS53YL_Vertical" H 9200 3300 50  0001 C CNN
 F 3 "~" H 9200 3300 50  0001 C CNN
 	1    9200 3300

Commit message: Add: Bauteiltypen Digikey...
viele Bauteile von WE da hoffentlich lange gueltig...
Parts:
- C701, C702, C703, C704, C707, C708, C709, C710, C711, C712, C713, C718, C725: Bauteil (none) -> WE 885382206004
- C705, C716, C717, C719, C720: Bauteil (none) -> WE 885012207078
- C706, C724: Bauteil (none) -> WE 885012208069
- C714, C715: Bauteil (none) -> WE 885012206079
- C721: Bauteil (none) -> WE 885012206093
- C722, C723: Bauteil (none) -> WE 885012206089
- L701: Bauteil (none) -> WE 744045004; Type WE 744045004 -> (none)
- RV701: value 22k lin -> 20k lin; footprint Potentiometer_SMD:Potentiometer_Vishay_TS53YL_Vertical -> Potentiometer_SMD:Potentiometer_Vishay_TS53YL_Vertica; Bauteil (none) -> Vishay TS53YL203MR10
- RV702: value 22k lin -> 20k lin; Bauteil (none) -> Vishay TS53YL203MR10
- U701: Bauteil (none) -> AD8656ARZ
- Y701: Bauteil (none) -> FC4SDCBMF12.288-T1
Connections:
- net Earth: now also C718.2; no longer C718.1
- net at R709.1, R710.1, R712.1: now also C718.1; no longer C718.2

Commit message: Change: Relais SMT -> THT, Sicherung PCB
Parts:
- RV701: footprint Potentiometer_SMD:Potentiometer_Vishay_TS53YL_Vertica -> Potentiometer_SMD:Potentiometer_Vishay_TS53YL_Vertical
- U702: Bauteil (none) -> VLSI VS1053B
Changed lines of the file:
@@
 encoding utf-8
 Sheet 7 7
-Title "Fernbedienung SABA 6-3D"
-Date "2021-01-13"
+Title "Fernbedienung - Webradio SABA 6-3D"
+Date "2021-01-14"
 Rev "1-A"
 Comp "Martin Wagner DL2WAG"
@@
 Comment2 "Audio"
 Comment3 "(Meersburg/Freiburg 6-3D, weitere?)"
-Comment4 "Fernbedienung für SABA \"Automatic\" Radios"
+Comment4 "Fernbedienung - Webradio für SABA \"Automatic\" Radios"
 $EndDescr
 $Comp
@@
 F 2 "Package_QFP:LQFP-48_7x7mm_P0.5mm" H 3150 5450 50  0001 C CNN
 F 3 "" H 3150 5450 50  0001 C CNN
+F 4 "VLSI VS1053B" H 3150 5450 50  0001 C CNN "Bauteil"
 	1    3150 5450
 	1    0    0    -1
@@
 F 0 "RV701" H 9131 1496 50  0000 R CNN
 F 1 "20k lin" H 9131 1405 50  0000 R CNN
-F 2 "Potentiometer_SMD:Potentiometer_Vishay_TS53YL_Vertica" H 9200 1450 50  0001 C CNN
+F 2 "Potentiometer_SMD:Potentiometer_Vishay_TS53YL_Vertical" H 9200 1450 50  0001 C CNN
 F 3 "~" H 9200 1450 50  0001 C CNN
 F 4 "Vishay TS53YL203MR10" H 9200 1450 50  0001 C CNN "Bauteil"

Commit message: Sicherung
Parts:
- Y701: Bauteil FC4SDCBMF12.288-T1 -> ABM3-12.288MHZ-D2Y-T
Changed lines of the file:
@@
 F 2 "Crystal:Crystal_SMD_HC49-SD" H 5300 3100 50  0001 C CNN
 F 3 "~" H 5300 3100 50  0001 C CNN
-F 4 "FC4SDCBMF12.288-T1" V 5300 3100 50  0001 C CNN "Bauteil"
+F 4 "ABM3-12.288MHZ-D2Y-T" V 5300 3100 50  0001 C CNN "Bauteil"
 	1    5300 3100
 	0    1    1    0

Commit message: PCB: Alle Leitungen verlegt
Connections:
- net Earth renamed GND
