File: cad/pcb/saba-fernbedienung/rev1-a/4-suchlauf-in.sch (KiCad schematic (older format))
At the start: 56 parts, among them U501 ADA4522-2, U502 LM339, U503 LTV-357T, U504 LTV-357T, U505 LTV-357T

Commit message: Fix: Div. DRC
Connections:
- net SABA_GND_AC: now also R535.2
- net at R528.2, R533.2, R534.1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: now also R535.1
- no-connect marks 0 -> 1
Changed lines of the file:
@@
 	2600 6850 2500 6850
 Wire Wire Line
-	2200 6850 1700 6850
+	2200 6850 2000 6850
 Connection ~ 1700 6850
 Wire Wire Line
@@
 Connection ~ 3050 6350
 Wire Wire Line
-	3150 7350 1700 7350
+	3150 7350 2000 7350
 Connection ~ 1700 7350
 $Comp
@@
 Wire Wire Line
 	7250 4950 6950 4950
+Connection ~ 2000 6850
+Wire Wire Line
+	2000 6850 1700 6850
+Connection ~ 2000 7350
+Wire Wire Line
+	2000 7350 1700 7350
+NoConn ~ 8100 5950
 $EndSCHEMATC

Commit message: New: Bauteil - Pad Zuordnungen
Parts:
- D501, D502: value D -> 1N4148; footprint (none) -> Diode_SMD:D_SOD-323F
- D503, D504: footprint (none) -> Diode_SMD:D_SMA
- U501: footprint (none) -> Package_SO:SOIC-8_3.9x4.9mm_P1.27mm
- U502: footprint (none) -> Package_SO:SOIC-14_3.9x8.7mm_P1.27mm
Changed lines of the file:
@@
 F 0 "U501" H 10008 1646 50  0000 L CNN
 F 1 "ADA4522-2" H 10000 1800 50  0000 L CNN
-F 2 "" H 10050 1600 50  0001 C CNN
+F 2 "Package_SO:SOIC-8_3.9x4.9mm_P1.27mm" H 10050 1600 50  0001 C CNN
 F 3 "https://www.analog.com/media/en/technical-documentation/data-sheets/ADA4522-1_4522-2_4522-4.pdf" H 10050 1600 50  0001 C CNN
 	3    10050 1600
@@
 F 0 "D504" V 1804 2330 50  0000 L CNN
 F 1 "SMAJ33CA" V 1895 2330 50  0000 L CNN
-F 2 "" H 1850 2250 50  0001 C CNN
+F 2 "Diode_SMD:D_SMA" H 1850 2250 50  0001 C CNN
 F 3 "~" H 1850 2250 50  0001 C CNN
 	1    1850 2250
@@
 AR Path="/60135668/60180DAE" Ref="D501"  Part="1"
 F 0 "D501" H 8500 1533 50  0000 C CNN
-F 1 "D" H 8500 1624 50  0000 C CNN
-F 2 "" H 8500 1750 50  0001 C CNN
+F 1 "1N4148" H 8500 1624 50  0000 C CNN
+F 2 "Diode_SMD:D_SOD-323F" H 8500 1750 50  0001 C CNN
 F 3 "~" H 8500 1750 50  0001 C CNN
 	1    8500 1750
@@
 F 0 "D503" V 6354 2280 50  0000 L CNN
 F 1 "SMAJ33CA" V 6445 2280 50  0000 L CNN
-F 2 "" H 6400 2200 50  0001 C CNN
+F 2 "Diode_SMD:D_SMA" H 6400 2200 50  0001 C CNN
 F 3 "~" H 6400 2200 50  0001 C CNN
 	1    6400 2200
@@
 AR Path="/60135668/60158950" Ref="D502"  Part="1"
 F 0 "D502" H 4500 1583 50  0000 C CNN
-F 1 "D" H 4500 1674 50  0000 C CNN
-F 2 "" H 4500 1800 50  0001 C CNN
+F 1 "1N4148" H 4500 1674 50  0000 C CNN
+F 2 "Diode_SMD:D_SOD-323F" H 4500 1800 50  0001 C CNN
 F 3 "~" H 4500 1800 50  0001 C CNN
 	1    4500 1800
@@
 F 0 "U501" H 7450 1383 50  0000 C CNN
 F 1 "ADA4522-2" H 7450 1474 50  0000 C CNN
-F 2 "" H 7450 1750 50  0001 C CNN
+F 2 "Package_SO:SOIC-8_3.9x4.9mm_P1.27mm" H 7450 1750 50  0001 C CNN
 F 3 "https://www.analog.com/media/en/technical-documentation/data-sheets/ADA4522-1_4522-2_4522-4.pdf" H 7450 1750 50  0001 C CNN
 	2    7450 1750
@@
 F 0 "U501" H 2500 1433 50  0000 C CNN
 F 1 "ADA4522-2" H 2500 1524 50  0000 C CNN
-F 2 "" H 2500 1800 50  0001 C CNN
+F 2 "Package_SO:SOIC-8_3.9x4.9mm_P1.27mm" H 2500 1800 50  0001 C CNN
 F 3 "https://www.analog.com/media/en/technical-documentation/data-sheets/ADA4522-1_4522-2_4522-4.pdf" H 2500 1800 50  0001 C CNN
 	1    2500 1800
@@
 F 0 "U502" H 2150 3583 50  0000 C CNN
 F 1 "LM339" H 2150 3674 50  0000 C CNN
-F 2 "" H 2100 4050 50  0001 C CNN
+F 2 "Package_SO:SOIC-14_3.9x8.7mm_P1.27mm" H 2100 4050 50  0001 C CNN
 F 3 "https://www.st.com/resource/en/datasheet/lm139.pdf" H 2200 4150 50  0001 C CNN
 	1    2150 3950
@@
 F 0 "U502" H 2150 5983 50  0000 C CNN
 F 1 "LM339" H 2150 6074 50  0000 C CNN
-F 2 "" H 2100 6450 50  0001 C CNN
+F 2 "Package_SO:SOIC-14_3.9x8.7mm_P1.27mm" H 2100 6450 50  0001 C CNN
 F 3 "https://www.st.com/resource/en/datasheet/lm139.pdf" H 2200 6550 50  0001 C CNN
 	2    2150 6350
@@
 F 0 "U502" H 7400 3583 50  0000 C CNN
 F 1 "LM339" H 7400 3674 50  0000 C CNN
-F 2 "" H 7350 4050 50  0001 C CNN
+F 2 "Package_SO:SOIC-14_3.9x8.7mm_P1.27mm" H 7350 4050 50  0001 C CNN
 F 3 "https://www.st.com/resource/en/datasheet/lm139.pdf" H 7450 4150 50  0001 C CNN
 	3    7400 3950
@@
 F 0 "U502" H 7800 5583 50  0000 C CNN
 F 1 "LM339" H 7800 5674 50  0000 C CNN
-F 2 "" H 7750 6050 50  0001 C CNN
+F 2 "Package_SO:SOIC-14_3.9x8.7mm_P1.27mm" H 7750 6050 50  0001 C CNN
 F 3 "https://www.st.com/resource/en/datasheet/lm139.pdf" H 7850 6150 50  0001 C CNN
 	4    7800 5950
@@
 F 0 "U502" H 10808 1646 50  0000 L CNN
 F 1 "LM339" H 10800 1800 50  0000 L CNN
-F 2 "" H 10800 1700 50  0001 C CNN
+F 2 "Package_SO:SOIC-14_3.9x8.7mm_P1.27mm" H 10800 1700 50  0001 C CNN
 F 3 "https://www.st.com/resource/en/datasheet/lm139.pdf" H 10900 1800 50  0001 C CNN
 	5    10850 1600

Commit message: Add: Bauteiltypen Digikey...
viele Bauteile von WE da hoffentlich lange gueltig...
Parts:
- C501, C502, C506, C507, C508: Bauteil (none) -> WE 885382206004
- C503, C504, C505: footprint Capacitor_SMD:C_0603_1608Metric -> Capacitor_SMD:C_0805_2012Metric; Bauteil (none) -> 885012207102
- D501, D502: Bauteil (none) -> ON 1N4148WS
- D503, D504: Bauteil (none) -> Diodes SMAJ33CAQ-13-F
- D505, D506, D507: Bauteil (none) -> WE 150080BS75000
- U501: Bauteil (none) -> ADA4522-1ARMZ
- U502: Bauteil (none) -> ON LM339DR2G
- U502: Bauteil (none) -> LM339DR2G
- U503, U504, U505: Bauteil (none) -> Lite-On LTV-357T
Changed lines of the file:
@@
 F 2 "Package_SO:SOIC-8_3.9x4.9mm_P1.27mm" H 10050 1600 50  0001 C CNN
 F 3 "https://www.analog.com/media/en/technical-documentation/data-sheets/ADA4522-1_4522-2_4522-4.pdf" H 10050 1600 50  0001 C CNN
+F 4 "ADA4522-1ARMZ" H 10050 1600 50  0001 C CNN "Bauteil"
 	3    10050 1600
 	1    0    0    -1
@@
 F 2 "Diode_SMD:D_SMA" H 1850 2250 50  0001 C CNN
 F 3 "~" H 1850 2250 50  0001 C CNN
+F 4 "Diodes SMAJ33CAQ-13-F" V 1850 2250 50  0001 C CNN "Bauteil"
 	1    1850 2250
 	0    1    1    0
@@
 F 2 "Diode_SMD:D_SOD-323F" H 8500 1750 50  0001 C CNN
 F 3 "~" H 8500 1750 50  0001 C CNN
+F 4 "ON 1N4148WS" H 8500 1750 50  0001 C CNN "Bauteil"
 	1    8500 1750
-	-1   0    0    1
-$EndComp
-$Comp
-L Device:C C?
-U 1 1 60180DA8
-P 8800 2050
-AR Path="/6002EA57/60180DA8" Ref="C?"  Part="1"
-AR Path="/6008B538/60180DA8" Ref="C?"  Part="1"
-AR Path="/60135668/60180DA8" Ref="C504"  Part="1"
-F 0 "C504" H 8915 2141 50  0000 L CNN
-F 1 "470n" H 8915 2050 50  0000 L CNN
-F 2 "Capacitor_SMD:C_0603_1608Metric" H 8838 1900 50  0001 C CNN
-F 3 "~" H 8800 2050 50  0001 C CNN
-F 4 "" H 8915 1959 50  0000 L CNN "Placement"
-	1    8800 2050
 	-1   0    0    1
 $EndComp
@@
 F 2 "Diode_SMD:D_SMA" H 6400 2200 50  0001 C CNN
 F 3 "~" H 6400 2200 50  0001 C CNN
+F 4 "Diodes SMAJ33CAQ-13-F" V 6400 2200 50  0001 C CNN "Bauteil"
 	1    6400 2200
 	0    1    1    0
@@
 	4800 2400 3650 2400
 Wire Wire Line
-	4800 2250 4800 2400
-Wire Wire Line
 	4800 1800 4800 1950
 Wire Wire Line
@@
 F 2 "Diode_SMD:D_SOD-323F" H 4500 1800 50  0001 C CNN
 F 3 "~" H 4500 1800 50  0001 C CNN
+F 4 "ON 1N4148WS" H 4500 1800 50  0001 C CNN "Bauteil"
 	1    4500 1800
-	-1   0    0    1
-$EndComp
-$Comp
-L Device:C C?
-U 1 1 6015830E
-P 4800 2100
-AR Path="/6002EA57/6015830E" Ref="C?"  Part="1"
-AR Path="/6008B538/6015830E" Ref="C?"  Part="1"
-AR Path="/60135668/6015830E" Ref="C505"  Part="1"
-F 0 "C505" H 4915 2191 50  0000 L CNN
-F 1 "470n" H 4915 2100 50  0000 L CNN
-F 2 "Capacitor_SMD:C_0603_1608Metric" H 4838 1950 50  0001 C CNN
-F 3 "~" H 4800 2100 50  0001 C CNN
-F 4 "" H 4915 2009 50  0000 L CNN "Placement"
-	1    4800 2100
 	-1   0    0    1
 $EndComp
@@
 F 0 "C503" H 3315 1891 50  0000 L CNN
 F 1 "470n" H 3315 1800 50  0000 L CNN
-F 2 "Capacitor_SMD:C_0603_1608Metric" H 3238 1650 50  0001 C CNN
+F 2 "Capacitor_SMD:C_0805_2012Metric" H 3238 1650 50  0001 C CNN
 F 3 "~" H 3200 1800 50  0001 C CNN
 F 4 "" H 3315 1709 50  0000 L CNN "Placement"
+F 5 "885012207102" H 3200 1800 50  0001 C CNN "Bauteil"
 	1    3200 1800
 	0    1    1    0
@@
 F 2 "Package_SO:SOIC-8_3.9x4.9mm_P1.27mm" H 7450 1750 50  0001 C CNN
 F 3 "https://www.analog.com/media/en/technical-documentation/data-sheets/ADA4522-1_4522-2_4522-4.pdf" H 7450 1750 50  0001 C CNN
+F 4 "ADA4522-1ARMZ" H 7450 1750 50  0001 C CNN "Bauteil"
 	2    7450 1750
 	1    0    0    1
@@
 F 2 "Package_SO:SOIC-8_3.9x4.9mm_P1.27mm" H 2500 1800 50  0001 C CNN
 F 3 "https://www.analog.com/media/en/technical-documentation/data-sheets/ADA4522-1_4522-2_4522-4.pdf" H 2500 1800 50  0001 C CNN
+F 4 "ADA4522-1ARMZ" H 2500 1800 50  0001 C CNN "Bauteil"
 	1    2500 1800
 	1    0    0    1
@@
 F 2 "Package_SO:SOIC-14_3.9x8.7mm_P1.27mm" H 2100 4050 50  0001 C CNN
 F 3 "https://www.st.com/resource/en/datasheet/lm139.pdf" H 2200 4150 50  0001 C CNN
+F 4 "ON LM339DR2G" H 2150 3950 50  0001 C CNN "Bauteil"
 	1    2150 3950
 	1    0    0    1
@@
 F 2 "Package_SO:SOIC-14_3.9x8.7mm_P1.27mm" H 2100 6450 50  0001 C CNN
 F 3 "https://www.st.com/resource/en/datasheet/lm139.pdf" H 2200 6550 50  0001 C CNN
+F 4 "LM339DR2G" H 2150 6350 50  0001 C CNN "Bauteil"
 	2    2150 6350
 	1    0    0    1
@@
 F 2 "Package_SO:SOIC-14_3.9x8.7mm_P1.27mm" H 7350 4050 50  0001 C CNN
 F 3 "https://www.st.com/resource/en/datasheet/lm139.pdf" H 7450 4150 50  0001 C CNN
+F 4 "LM339DR2G" H 7400 3950 50  0001 C CNN "Bauteil"
 	3    7400 3950
 	1    0    0    1
@@
 F 2 "Package_SO:SOIC-14_3.9x8.7mm_P1.27mm" H 7750 6050 50  0001 C CNN
 F 3 "https://www.st.com/resource/en/datasheet/lm139.pdf" H 7850 6150 50  0001 C CNN
+F 4 "LM339DR2G" H 7800 5950 50  0001 C CNN "Bauteil"
 	4    7800 5950
 	1    0    0    1
@@
 F 2 "Package_SO:SOIC-14_3.9x8.7mm_P1.27mm" H 10800 1700 50  0001 C CNN
 F 3 "https://www.st.com/resource/en/datasheet/lm139.pdf" H 10900 1800 50  0001 C CNN
+F 4 "LM339DR2G" H 10850 1600 50  0001 C CNN "Bauteil"
 	5    10850 1600
 	1    0    0    -1
@@
 F 2 "Package_SO:SO-4_4.4x3.6mm_P2.54mm" H 3250 3850 50  0001 L CIN
 F 3 "https://www.buerklin.com/medias/sys_master/download/download/h91/ha0/8892020588574.pdf" H 3450 4050 50  0001 L CNN
+F 4 "Lite-On LTV-357T" H 3450 4050 50  0001 C CNN "Bauteil"
 	1    3450 4050
 	1    0    0    -1
@@
 F 3 "~" H 4500 4200 50  0001 C CNN
 F 4 "" H 4615 4109 50  0000 L CNN "Placement"
+F 5 "WE 885382206004" H 4500 4200 50  0001 C CNN "Bauteil"
 	1    4500 4200
 	-1   0    0    1
@@
 F 2 "Package_SO:SO-4_4.4x3.6mm_P2.54mm" H 3250 6250 50  0001 L CIN
 F 3 "https://www.buerklin.com/medias/sys_master/download/download/h91/ha0/8892020588574.pdf" H 3450 6450 50  0001 L CNN
+F 4 "Lite-On LTV-357T" H 3450 6450 50  0001 C CNN "Bauteil"
 	1    3450 6450
 	1    0    0    -1
@@
 F 3 "~" H 4500 6600 50  0001 C CNN
 F 4 "" H 4615 6509 50  0000 L CNN "Placement"
+F 5 "WE 885382206004" H 4500 6600 50  0001 C CNN "Bauteil"
 	1    4500 6600
 	-1   0    0    1
@@
 F 2 "Package_SO:SO-4_4.4x3.6mm_P2.54mm" H 8500 3850 50  0001 L CIN
 F 3 "https://www.buerklin.com/medias/sys_master/download/download/h91/ha0/8892020588574.pdf" H 8700 4050 50  0001 L CNN
+F 4 "Lite-On LTV-357T" H 8700 4050 50  0001 C CNN "Bauteil"
 	1    8700 4050
 	1    0    0    -1
@@
 F 3 "~" H 9750 4200 50  0001 C CNN
 F 4 "" H 9865 4109 50  0000 L CNN "Placement"
+F 5 "WE 885382206004" H 9750 4200 50  0001 C CNN "Bauteil"
 	1    9750 4200
 	-1   0    0    1
@@
 F 3 "~" H 9700 1650 50  0001 C CNN
 F 4 "" H 9815 1559 50  0000 L CNN "Placement"
+F 5 "WE 885382206004" H 9700 1650 50  0001 C CNN "Bauteil"
 	1    9700 1650
 	-1   0    0    1
@@
 F 3 "~" H 10500 1650 50  0001 C CNN
 F 4 "" H 10615 1559 50  0000 L CNN "Placement"
+F 5 "WE 885382206004" H 10500 1650 50  0001 C CNN "Bauteil"
 	1    10500 1650
 	-1   0    0    1
@@
 F 2 "LED_SMD:LED_0805_2012Metric" H 3150 4350 50  0001 C CNN
 F 3 "~" H 3150 4350 50  0001 C CNN
+F 4 "WE 150080BS75000" V 3150 4350 50  0001 C CNN "Bauteil"
 	1    3150 4350
 	0    -1   -1   0
@@
 F 2 "LED_SMD:LED_0805_2012Metric" H 3150 6750 50  0001 C CNN
 F 3 "~" H 3150 6750 50  0001 C CNN
+F 4 "WE 150080BS75000" V 3150 6750 50  0001 C CNN "Bauteil"
 	1    3150 6750
 	0    -1   -1   0
@@
 F 2 "LED_SMD:LED_0805_2012Metric" H 8400 4350 50  0001 C CNN
 F 3 "~" H 8400 4350 50  0001 C CNN
+F 4 "WE 150080BS75000" V 8400 4350 50  0001 C CNN "Bauteil"
 	1    8400 4350
 	0    -1   -1   0
@@
 	2000 7350 1700 7350
 NoConn ~ 8100 5950
+$Comp
+L Device:C C?
+U 1 1 600521DF
+P 8800 2050
+AR Path="/6002EA57/600521DF" Ref="C?"  Part="1"
+AR Path="/6008B538/600521DF" Ref="C?"  Part="1"
+AR Path="/60135668/600521DF" Ref="C504"  Part="1"
+F 0 "C504" H 8915 2141 50  0000 L CNN
+F 1 "470n" H 8915 2050 50  0000 L CNN
+F 2 "Capacitor_SMD:C_0805_2012Metric" H 8838 1900 50  0001 C CNN
+F 3 "~" H 8800 2050 50  0001 C CNN
+F 4 "" H 8915 1959 50  0000 L CNN "Placement"
+F 5 "885012207102" H 8800 2050 50  0001 C CNN "Bauteil"
+	1    8800 2050
+	-1   0    0    1
+$EndComp
+Wire Wire Line
+	4800 2250 4800 2400
+$Comp
+L Device:C C?
+U 1 1 600539D8
+P 4800 2100
+AR Path="/6002EA57/600539D8" Ref="C?"  Part="1"
+AR Path="/6008B538/600539D8" Ref="C?"  Part="1"
+AR Path="/60135668/600539D8" Ref="C505"  Part="1"
+F 0 "C505" H 4915 2191 50  0000 L CNN
+F 1 "470n" H 4915 2100 50  0000 L CNN
+F 2 "Capacitor_SMD:C_0805_2012Metric" H 4838 1950 50  0001 C CNN
+F 3 "~" H 4800 2100 50  0001 C CNN
+F 4 "" H 4915 2009 50  0000 L CNN "Placement"
+F 5 "885012207102" H 4800 2100 50  0001 C CNN "Bauteil"
+	1    4800 2100
+	-1   0    0    1
+$EndComp
 $EndSCHEMATC

Commit message: Change: Relais SMT -> THT, Sicherung PCB
Parts:
- C503, C504, C505: Bauteil 885012207102 -> WE 885012207102
Changed lines of the file:
@@
 encoding utf-8
 Sheet 5 7
-Title "Fernbedienung SABA 6-3D"
-Date "2021-01-13"
+Title "Fernbedienung - Webradio SABA 6-3D"
+Date "2021-01-14"
 Rev "1-A"
 Comp "Martin Wagner DL2WAG"
@@
 Comment2 "Suchlauf Eingang"
 Comment3 "(Meersburg/Freiburg 6-3D, weitere?)"
-Comment4 "Fernbedienung für SABA \"Automatic\" Radios"
+Comment4 "Fernbedienung - Webradio für SABA \"Automatic\" Radios"
 $EndDescr
 Text Notes 650  800  0    79   ~ 0
@@
 F 3 "~" H 3200 1800 50  0001 C CNN
 F 4 "" H 3315 1709 50  0000 L CNN "Placement"
-F 5 "885012207102" H 3200 1800 50  0001 C CNN "Bauteil"
+F 5 "WE 885012207102" H 3200 1800 50  0001 C CNN "Bauteil"
 	1    3200 1800
 	0    1    1    0
@@
 F 3 "~" H 8800 2050 50  0001 C CNN
 F 4 "" H 8915 1959 50  0000 L CNN "Placement"
-F 5 "885012207102" H 8800 2050 50  0001 C CNN "Bauteil"
+F 5 "WE 885012207102" H 8800 2050 50  0001 C CNN "Bauteil"
 	1    8800 2050
 	-1   0    0    1
@@
 F 3 "~" H 4800 2100 50  0001 C CNN
 F 4 "" H 4915 2009 50  0000 L CNN "Placement"
-F 5 "885012207102" H 4800 2100 50  0001 C CNN "Bauteil"
+F 5 "WE 885012207102" H 4800 2100 50  0001 C CNN "Bauteil"
 	1    4800 2100
 	-1   0    0    1

Commit message: Fix: Opamp zweifach
Parts:
- U501: Bauteil ADA4522-1ARMZ -> ADA4522-2ARMZ
Changed lines of the file:
@@
 F 2 "Package_SO:SOIC-8_3.9x4.9mm_P1.27mm" H 2500 1800 50  0001 C CNN
 F 3 "https://www.analog.com/media/en/technical-documentation/data-sheets/ADA4522-1_4522-2_4522-4.pdf" H 2500 1800 50  0001 C CNN
-F 4 "ADA4522-1ARMZ" H 2500 1800 50  0001 C CNN "Bauteil"
+F 4 "ADA4522-2ARMZ" H 2500 1800 50  0001 C CNN "Bauteil"
 	1    2500 1800
 	1    0    0    1
