File: cad/pcb/saba-fernbedienung/rev1-a/saba-fernbedienung.kicad_pcb (KiCad board)
At the start: 4 copper layers, 100 x 81.8 mm, 236 parts, among them J201 Conn_ARM_JTAG_SWD_10, J301 Conn_01x04, J302 Conn_01x04, J303 Micro_SD_Card, J304 Conn_01x04, J305 AudioJack3, J306 Conn_01x02, J307 Conn_01x04, J308 Conn_01x01, J309 Conn_01x01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

Commit message: Add: Herstellungsdaten
Routing:
- removed copper zone on B.Cu, net -24V
Other:
- outline, holes or cut-outs redrawn
