File: cad/pcb/saba-fernbedienung-anschlussstecker/rev1-a/saba-fernbedienung-anschlussstecker.kicad_pcb (KiCad board)
At the start: 2 copper layers, 38.5 x 39.1 mm, 8 parts, among them J101 Conn_01x04, J102 Conn_01x04, J103 Conn_01x04, J104 Conn_01x02, J105 Conn_01x04, J106 Conn_01x04, X101 Stecker-6-3D

Commit message: Change: Position Steckerpins
Routing:
- net Net-(J102-Pad3): track 13.2 -> 11.5 mm
Other:
- outline, holes or cut-outs redrawn

Commit message: Add: Herstellungsdaten
Other:
- outline, holes or cut-outs redrawn
