File: cad/pcb/saba-fernbedienung/rev2-a/1-microcontroller.sch (KiCad schematic (older format))
At the start: 10 parts, among them J201 Conn_ARM_JTAG_SWD_10, Q201 BC856, U201 DOIT-DEVKITV1-ESP32-WROOM-32

Commit message: ToDo-s bearbeitet
Parts:
- removed D201: LED, LED_SMD:LED_0805_2012Metric, symbol Device:LED
- removed Q201: BC856, Package_TO_SOT_SMD:SOT-23, symbol Transistor_BJT:BC856
- removed R203: 10k, Resistor_SMD:R_0603_1608Metric, symbol Device:R
- removed R204: 1k, Resistor_SMD:R_0603_1608Metric, symbol Device:R
- added D?: 1N4148, Diode_SMD:D_SOD-323F, symbol Device:D
- added R?: 10k, Resistor_SMD:R_0603_1608Metric, symbol Device:R
- added R?: 0, Resistor_SMD:R_0603_1608Metric, symbol Device:R
Connections:
- net LCD_A0 is gone; now on net SPI_MOSI: U201.15 (IO23)
- net +3V3: now also R?.2
- net SABA_Laut: now also R206.2, U201.3 (IO15); no longer U201.4 (IO2)
- net SABA_Leise: now also U201.4 (IO2); no longer R206.2, U201.3 (IO15)
- net SABA_Suchlauf_L: now also R208.2, U201.28 (IO13); no longer R207.2, U201.26 (IO14)
- net SABA_Suchlauf_R: now also R207.2, U201.26 (IO14); no longer R208.2, U201.28 (IO13)
- net SPI_MOSI: no longer U201.11 (IO21)
- net ~RESET: now also D?.2 (A), R?.1, R?.2; no longer U201.16 (EN/~RESET)
- net at U201.7 (IO17): now also R?.1
- net TA_Aktiv: now reaches U201.18 (SENSOR_VN/IO39)
- net SABA_Netz renamed SABA_Netz_Set
- net SPI_CS_LCD renamed SABA_Netz_Reset
- new net: D?.1 (K), U201.16 (EN/~RESET)
- new net SABA_Netz_Feedback: U201.11 (IO21)
Changed lines of the file:
@@
 Sheet 2 7
 Title "Fernbedienung - Webradio SABA 6-3D"
-Date "2021-01-16"
-Rev "1-A"
+Date "2021-08-14"
+Rev "2-A"
 Comp "Martin Wagner DL2WAG"
 Comment1 "Lizenz: CERN-OHL-W (OHL v2)"
@@
 Comment4 "Fernbedienung - Webradio für SABA \"Automatic\" Radios"
 $EndDescr
-Text GLabel 1700 1900 0    50   BiDi ~ 0
+Text GLabel 1250 1900 0    50   Output ~ 0
 ~RESET
 Wire Wire Line
-	1700 1900 2100 1900
+	1950 1900 2100 1900
 $Comp
 L power:GND #PWR0206
@@
 Text GLabel 5550 3000 2    50   Input ~ 0
 SPI_MISO
-Text GLabel 5550 3100 2    50   Output ~ 0
-SPI_MOSI
-Wire Wire Line
-	5550 3100 3300 3100
 Wire Wire Line
 	3300 3000 5550 3000
@@
 Wire Wire Line
 	5550 3700 3300 3700
-Text GLabel 5550 3300 2    50   BiDi ~ 0
-LCD_A0
-Text GLabel 5550 3400 2    50   Output ~ 0
-SPI_CS_LCD
 Text GLabel 5550 3200 2    50   Output ~ 0
 SPI_CS_SDCARD
@@
 Wire Wire Line
 	5550 4000 3300 4000
-$Comp
-L Device:R R203
-U 1 1 5FFDB025
-P 7850 2800
-F 0 "R203" V 7650 2800 50  0000 C CNN
-F 1 "10k" V 7750 2800 50  0000 C CNN
-F 2 "Resistor_SMD:R_0603_1608Metric" V 7780 2800 50  0001 C CNN
-F 3 "~" H 7850 2800 50  0001 C CNN
-F 4 "NP" V 7850 2800 50  0000 C CNN "Placement"
-	1    7850 2800
-	0    1    1    0
-$EndComp
-Wire Wire Line
-	7700 2800 3300 2800
-Wire Wire Line
-	8100 2800 8000 2800
-Wire Wire Line
-	8400 3000 8400 3200
-Wire Wire Line
-	8400 3200 8850 3200
-Text GLabel 8850 3200 2    50   Output ~ 0
-LCD_BL
-$Comp
-L power:+3V3 #PWR0203
-U 1 1 5FFE05B3
-P 8400 2500
-F 0 "#PWR0203" H 8400 2350 50  0001 C CNN
-F 1 "+3V3" H 8415 2673 50  0000 C CNN
-F 2 "" H 8400 2500 50  0001 C CNN
-F 3 "" H 8400 2500 50  0001 C CNN
-	1    8400 2500
-	1    0    0    -1
-$EndComp
-Wire Wire Line
-	8400 2500 8400 2600
 Text GLabel 5550 4100 2    50   Input ~ 0
 SABA_HS
 Wire Wire Line
 	5550 3900 3300 3900
+Text GLabel 5550 2500 2    50   Output ~ 0
+SABA_Suchlauf_R
 Text GLabel 5550 2400 2    50   Output ~ 0
-SABA_Suchlauf_R
-Text GLabel 5550 2500 2    50   Output ~ 0
 SABA_Suchlauf_L
 Wire Wire Line
@@
 Text GLabel 5550 2700 2    50   Output ~ 0
 SABA_Mute
-Text GLabel 5550 1900 2    50   Output ~ 0
-SABA_Laut
-Text GLabel 5550 2600 2    50   Output ~ 0
-SABA_Leise
 Text GLabel 5550 3500 2    50   Output ~ 0
-SABA_Netz
+SABA_Netz_Set
 Text GLabel 5550 3600 2    50   Input ~ 0
 SABA_Laufrichtung
@@
 Text GLabel 5550 3900 2    50   Input ~ 0
 SABA_Suchlauf_Schnell
-$Comp
-L Device:R R204
-U 1 1 5FFF2B18
-P 3550 4450
-F 0 "R204" H 3480 4404 50  0000 R CNN
-F 1 "1k" H 3480 4495 50  0000 R CNN
-F 2 "Resistor_SMD:R_0603_1608Metric" V 3480 4450 50  0001 C CNN
-F 3 "~" H 3550 4450 50  0001 C CNN
-F 4 "" V 3435 4450 50  0001 C CNN "Placement"
-	1    3550 4450
-	-1   0    0    1
-$EndComp
-Wire Wire Line
-	5550 3300 3300 3300
 Wire Wire Line
 	5550 3400 3300 3400
@@
 Wire Wire Line
 	5550 4100 3300 4100
-Wire Wire Line
-	3550 4300 3550 4200
-Wire Wire Line
-	3550 4200 3300 4200
-$Comp
-L power:GND #PWR0208
-U 1 1 5FFF784B
-P 3550 5050
-F 0 "#PWR0208" H 3550 4800 50  0001 C CNN
-F 1 "GND" H 3555 4877 50  0000 C CNN
-F 2 "" H 3550 5050 50  0001 C CNN
-F 3 "" H 3550 5050 50  0001 C CNN
-	1    3550 5050
-	1    0    0    -1
-$EndComp
-$Comp
-L Device:LED D201
-U 1 1 5FFF97AB
-P 3550 4800
-F 0 "D201" V 3589 4682 50  0000 R CNN
-F 1 "LED" V 3498 4682 50  0000 R CNN
-F 2 "LED_SMD:LED_0805_2012Metric" H 3550 4800 50  0001 C CNN
-F 3 "~" H 3550 4800 50  0001 C CNN
-F 4 "WE 150080BS75000" V 3550 4800 50  0001 C CNN "Bauteil"
-	1    3550 4800
-	0    -1   -1   0
-$EndComp
-Wire Wire Line
-	3550 4600 3550 4650
-Wire Wire Line
-	3550 4950 3550 5050
 $Comp
 L Connector:Conn_ARM_JTAG_SWD_10 J201
@@
 	4550 2500 5550 2500
 Connection ~ 4550 2500
-$Comp
-L Transistor_BJT:BC856 Q201
-U 1 1 5FFDE545
-P 8300 2800
-F 0 "Q201" H 8491 2709 50  0000 L CNN
-F 1 "BC856" H 8491 2800 50  0000 L CNN
-F 2 "Package_TO_SOT_SMD:SOT-23" H 8500 2725 50  0001 L CIN
-F 3 "" H 8300 2800 50  0001 L CNN
-F 4 "NP" H 8491 2891 50  0000 L CNN "Placement"
-F 5 "ON BC856BLT1G" H 8300 2800 50  0001 C CNN "Bauteil"
-	1    8300 2800
-	1    0    0    1
-$EndComp
 Wire Wire Line
 	5550 2700 3300 2700
 NoConn ~ 3300 2000
+Text GLabel 5550 3300 2    50   Output ~ 0
+SPI_MOSI
+Wire Wire Line
+	5550 3300 3300 3300
+Text GLabel 5550 1900 2    50   Output ~ 0
+SABA_Leise
+Text GLabel 5550 2600 2    50   Output ~ 0
+SABA_Laut
+Text GLabel 5550 3400 2    50   Output ~ 0
+SABA_Netz_Reset
+Text GLabel 5550 3100 2    50   Input ~ 0
+SABA_Netz_Feedback
+Wire Wire Line
+	5550 3100 3300 3100
+Wire Wire Line
+	1650 1900 1450 1900
+Text GLabel 5550 2800 2    50   Output ~ 0
+~RESET
+$Comp
+L Device:R R?
+U 1 1 61300578
+P 1450 1600
+F 0 "R?" H 1380 1554 50  0000 R CNN
+F 1 "10k" H 1380 1645 50  0000 R CNN
+F 2 "Resistor_SMD:R_0603_1608Metric" V 1380 1600 50  0001 C CNN
+F 3 "~" H 1450 1600 50  0001 C CNN
+F 4 "" V 1450 1600 50  0000 C CNN "Placement"
+	1    1450 1600
+	-1   0    0    1
+$EndComp
+$Comp
+L power:+3V3 #PWR?
+U 1 1 61300CA4
+P 1450 1350
+F 0 "#PWR?" H 1450 1200 50  0001 C CNN
+F 1 "+3V3" H 1465 1523 50  0000 C CNN
+F 2 "" H 1450 1350 50  0001 C CNN
+F 3 "" H 1450 1350 50  0001 C CNN
+	1    1450 1350
+	1    0    0    -1
+$EndComp
+Wire Wire Line
+	1450 1350 1450 1450
+Wire Wire Line
+	1450 1750 1450 1900
+Connection ~ 1450 1900
+Wire Wire Line
+	1450 1900 1250 1900
+$Comp
+L Device:R R?
+U 1 1 61303F4D
+P 5200 2800
+F 0 "R?" V 5150 3100 50  0000 R CNN
+F 1 "0" V 5150 2650 50  0000 R CNN
+F 2 "Resistor_SMD:R_0603_1608Metric" V 5130 2800 50  0001 C CNN
+F 3 "~" H 5200 2800 50  0001 C CNN
+F 4 "NP" V 5200 2850 50  0000 R CNN "Placement"
+	1    5200 2800
+	0    -1   -1   0
+$EndComp
+Wire Wire Line
+	5550 2800 5350 2800
+Wire Wire Line
+	5050 2800 3300 2800
+$Comp
+L Device:D D?
+U 1 1 612F9783
+P 1800 1900
+AR Path="/6008B538/612F9783" Ref="D?"  Part="1"
+AR Path="/60135668/612F9783" Ref="D?"  Part="1"
+AR Path="/5FFC49DA/612F9783" Ref="D?"  Part="1"
+F 0 "D?" H 1800 1683 50  0000 C CNN
+F 1 "1N4148" H 1800 1774 50  0000 C CNN
+F 2 "Diode_SMD:D_SOD-323F" H 1800 1900 50  0001 C CNN
+F 3 "~" H 1800 1900 50  0001 C CNN
+F 4 "0R" H 1800 1900 50  0001 C CNN "Bauteil"
+F 5 "" H 1800 2000 50  0001 C CNN "Placement"
+	1    1800 1900
+	-1   0    0    1
+$EndComp
+Text GLabel 5550 4200 2    50   Input ~ 0
+TA_Aktiv
+Wire Wire Line
+	3300 4200 5550 4200
 $EndSCHEMATC

Commit message: Change: Bauteilbezeichner
Parts:
- gave numbers to parts that had none: 3
- renumbered R205 to R203, R206 to R204, R207 to R205, R208 to R206
Changed lines of the file:
@@
 	1950 1900 2100 1900
 $Comp
-L power:GND #PWR0206
+L power:GND #PWR0205
 U 1 1 5FFCD50A
 P 2600 4750
-F 0 "#PWR0206" H 2600 4500 50  0001 C CNN
+F 0 "#PWR0205" H 2600 4500 50  0001 C CNN
 F 1 "GND" H 2605 4577 50  0000 C CNN
 F 2 "" H 2600 4750 50  0001 C CNN
@@
 $EndComp
 $Comp
-L power:GND #PWR0207
+L power:GND #PWR0206
 U 1 1 5FFCDB31
 P 2800 4750
-F 0 "#PWR0207" H 2800 4500 50  0001 C CNN
+F 0 "#PWR0206" H 2800 4500 50  0001 C CNN
 F 1 "GND" H 2805 4577 50  0000 C CNN
 F 2 "" H 2800 4750 50  0001 C CNN
@@
 	2800 4600 2800 4750
 $Comp
-L power:+3V3 #PWR0204
+L power:+3V3 #PWR0203
 U 1 1 5FFCE66A
 P 1900 2650
-F 0 "#PWR0204" H 1900 2500 50  0001 C CNN
+F 0 "#PWR0203" H 1900 2500 50  0001 C CNN
 F 1 "+3V3" H 1915 2823 50  0000 C CNN
 F 2 "" H 1900 2650 50  0001 C CNN
@@
 	1900 2750 2100 2750
 $Comp
-L power:+5V #PWR0201
+L power:+5V #PWR0202
 U 1 1 5FFD0017
 P 2700 1350
-F 0 "#PWR0201" H 2700 1200 50  0001 C CNN
+F 0 "#PWR0202" H 2700 1200 50  0001 C CNN
 F 1 "+5V" H 2715 1523 50  0000 C CNN
 F 2 "" H 2700 1350 50  0001 C CNN
@@
 ~RESET
 $Comp
-L power:+3V3 #PWR0205
+L power:+3V3 #PWR0204
 U 1 1 6001024E
 P 5750 4500
-F 0 "#PWR0205" H 5750 4350 50  0001 C CNN
+F 0 "#PWR0204" H 5750 4350 50  0001 C CNN
 F 1 "+3V3" H 5765 4673 50  0000 C CNN
 F 2 "" H 5750 4500 50  0001 C CNN
@@
 $EndComp
 $Comp
-L power:GND #PWR0209
+L power:GND #PWR0207
 U 1 1 60010E9A
 P 5750 5900
-F 0 "#PWR0209" H 5750 5650 50  0001 C CNN
+F 0 "#PWR0207" H 5750 5650 50  0001 C CNN
 F 1 "GND" H 5755 5727 50  0000 C CNN
 F 2 "" H 5750 5900 50  0001 C CNN
@@
 $EndComp
 $Comp
-L Device:R R205
+L Device:R R203
 U 1 1 6001163D
 P 3950 4450
-F 0 "R205" H 3900 4300 50  0000 R CNN
+F 0 "R203" H 3900 4300 50  0000 R CNN
 F 1 "100" H 3880 4450 50  0000 R CNN
 F 2 "Resistor_SMD:R_0603_1608Metric" V 3880 4450 50  0001 C CNN
@@
 $EndComp
 $Comp
-L Device:R R206
+L Device:R R204
 U 1 1 6001220B
 P 4250 4450
-F 0 "R206" H 4200 4300 50  0000 R CNN
+F 0 "R204" H 4200 4300 50  0000 R CNN
 F 1 "100" H 4180 4450 50  0000 R CNN
 F 2 "Resistor_SMD:R_0603_1608Metric" V 4180 4450 50  0001 C CNN
@@
 $EndComp
 $Comp
-L Device:R R208
+L Device:R R206
 U 1 1 60012608
 P 4850 4450
-F 0 "R208" H 4800 4300 50  0000 R CNN
+F 0 "R206" H 4800 4300 50  0000 R CNN
 F 1 "100" H 4780 4450 50  0000 R CNN
 F 2 "Resistor_SMD:R_0603_1608Metric" V 4780 4450 50  0001 C CNN
@@
 $EndComp
 $Comp
-L Device:R R207
+L Device:R R205
 U 1 1 60012995
 P 4550 4450
-F 0 "R207" H 4500 4300 50  0000 R CNN
+F 0 "R205" H 4500 4300 50  0000 R CNN
 F 1 "100" H 4480 4450 50  0000 R CNN
 F 2 "Resistor_SMD:R_0603_1608Metric" V 4480 4450 50  0001 C CNN
@@
 ~RESET
 $Comp
-L Device:R R?
+L Device:R R201
 U 1 1 61300578
 P 1450 1600
-F 0 "R?" H 1380 1554 50  0000 R CNN
+F 0 "R201" H 1380 1554 50  0000 R CNN
 F 1 "10k" H 1380 1645 50  0000 R CNN
 F 2 "Resistor_SMD:R_0603_1608Metric" V 1380 1600 50  0001 C CNN
@@
 $EndComp
 $Comp
-L power:+3V3 #PWR?
+L power:+3V3 #PWR0201
 U 1 1 61300CA4
 P 1450 1350
-F 0 "#PWR?" H 1450 1200 50  0001 C CNN
+F 0 "#PWR0201" H 1450 1200 50  0001 C CNN
 F 1 "+3V3" H 1465 1523 50  0000 C CNN
 F 2 "" H 1450 1350 50  0001 C CNN
@@
 	1450 1900 1250 1900
 $Comp
-L Device:R R?
+L Device:R R202
 U 1 1 61303F4D
 P 5200 2800
-F 0 "R?" V 5150 3100 50  0000 R CNN
+F 0 "R202" V 5150 3100 50  0000 R CNN
 F 1 "0" V 5150 2650 50  0000 R CNN
 F 2 "Resistor_SMD:R_0603_1608Metric" V 5130 2800 50  0001 C CNN
@@
 AR Path="/6008B538/612F9783" Ref="D?"  Part="1"
 AR Path="/60135668/612F9783" Ref="D?"  Part="1"
-AR Path="/5FFC49DA/612F9783" Ref="D?"  Part="1"
-F 0 "D?" H 1800 1683 50  0000 C CNN
+AR Path="/5FFC49DA/612F9783" Ref="D201"  Part="1"
+F 0 "D201" H 1800 1683 50  0000 C CNN
 F 1 "1N4148" H 1800 1774 50  0000 C CNN
 F 2 "Diode_SMD:D_SOD-323F" H 1800 1900 50  0001 C CNN

Commit message: Sicherung
Parts:
- added C201: 100n, Capacitor_SMD:C_0603_1608Metric, symbol Device:C
- added D202: 1N4148, Diode_SMD:D_SOD-323F, symbol Device:D
- added R203: 4k7, Resistor_SMD:R_0603_1608Metric, symbol Device:R
- added R204: 10k, Resistor_SMD:R_0603_1608Metric, symbol Device:R
- added R205: 1k, Resistor_SMD:R_0603_1608Metric, symbol Device:R
- added U202: LTV-357T, Package_SO:SO-4_4.4x3.6mm_P2.54mm, symbol Isolator:LTV-357T
- renumbered R203 to R206, R204 to R207, R205 to R208, R206 to R209
Connections:
- net +3V3: now also R203.1
- net GND: now also C201.1, U202.3
- net TA_Aktiv: now also D202.2 (A); no longer U201.18 (SENSOR_VN/IO39)
- new net: C201.2, R204.1, U201.18 (SENSOR_VN/IO39)
- new net: D202.1 (K), R205.1
- new net: R205.2, U202.1
- new net: R203.2, R204.2, U202.4
- new net Earth: U202.2
Changed lines of the file:
@@
 	1950 1900 2100 1900
 $Comp
-L power:GND #PWR0205
+L power:GND #PWR0209
 U 1 1 5FFCD50A
 P 2600 4750
-F 0 "#PWR0205" H 2600 4500 50  0001 C CNN
+F 0 "#PWR0209" H 2600 4500 50  0001 C CNN
 F 1 "GND" H 2605 4577 50  0000 C CNN
 F 2 "" H 2600 4750 50  0001 C CNN
@@
 $EndComp
 $Comp
-L power:GND #PWR0206
+L power:GND #PWR0210
 U 1 1 5FFCDB31
 P 2800 4750
-F 0 "#PWR0206" H 2800 4500 50  0001 C CNN
+F 0 "#PWR0210" H 2800 4500 50  0001 C CNN
 F 1 "GND" H 2805 4577 50  0000 C CNN
 F 2 "" H 2800 4750 50  0001 C CNN
@@
 ~RESET
 $Comp
-L power:+3V3 #PWR0204
+L power:+3V3 #PWR0205
 U 1 1 6001024E
 P 5750 4500
-F 0 "#PWR0204" H 5750 4350 50  0001 C CNN
+F 0 "#PWR0205" H 5750 4350 50  0001 C CNN
 F 1 "+3V3" H 5765 4673 50  0000 C CNN
 F 2 "" H 5750 4500 50  0001 C CNN
@@
 $EndComp
 $Comp
-L power:GND #PWR0207
+L power:GND #PWR0211
 U 1 1 60010E9A
 P 5750 5900
-F 0 "#PWR0207" H 5750 5650 50  0001 C CNN
+F 0 "#PWR0211" H 5750 5650 50  0001 C CNN
 F 1 "GND" H 5755 5727 50  0000 C CNN
 F 2 "" H 5750 5900 50  0001 C CNN
@@
 $EndComp
 $Comp
-L Device:R R203
+L Device:R R206
 U 1 1 6001163D
 P 3950 4450
-F 0 "R203" H 3900 4300 50  0000 R CNN
+F 0 "R206" H 3900 4300 50  0000 R CNN
 F 1 "100" H 3880 4450 50  0000 R CNN
 F 2 "Resistor_SMD:R_0603_1608Metric" V 3880 4450 50  0001 C CNN
@@
 $EndComp
 $Comp
-L Device:R R204
+L Device:R R207
 U 1 1 6001220B
 P 4250 4450
-F 0 "R204" H 4200 4300 50  0000 R CNN
+F 0 "R207" H 4200 4300 50  0000 R CNN
 F 1 "100" H 4180 4450 50  0000 R CNN
 F 2 "Resistor_SMD:R_0603_1608Metric" V 4180 4450 50  0001 C CNN
@@
 $EndComp
 $Comp
-L Device:R R206
+L Device:R R209
 U 1 1 60012608
 P 4850 4450
-F 0 "R206" H 4800 4300 50  0000 R CNN
+F 0 "R209" H 4800 4300 50  0000 R CNN
 F 1 "100" H 4780 4450 50  0000 R CNN
 F 2 "Resistor_SMD:R_0603_1608Metric" V 4780 4450 50  0001 C CNN
@@
 $EndComp
 $Comp
-L Device:R R205
+L Device:R R208
 U 1 1 60012995
 P 4550 4450
-F 0 "R205" H 4500 4300 50  0000 R CNN
+F 0 "R208" H 4500 4300 50  0000 R CNN
 F 1 "100" H 4480 4450 50  0000 R CNN
 F 2 "Resistor_SMD:R_0603_1608Metric" V 4480 4450 50  0001 C CNN
@@
 	-1   0    0    1
 $EndComp
-Text GLabel 5550 4200 2    50   Input ~ 0
+$Comp
+L Device:R R205
+U 1 1 618FB8CA
+P 9300 4200
+AR Path="/5FFC49DA/618FB8CA" Ref="R205"  Part="1"
+AR Path="/6002EA57/618FB8CA" Ref="R?"  Part="1"
+AR Path="/60135668/618FB8CA" Ref="R?"  Part="1"
+AR Path="/6044FE50/618FB8CA" Ref="R?"  Part="1"
+F 0 "R205" H 9230 4109 50  0000 R CNN
+F 1 "1k" H 9230 4200 50  0000 R CNN
+F 2 "Resistor_SMD:R_0603_1608Metric" V 9230 4200 50  0001 C CNN
+F 3 "~" H 9300 4200 50  0001 C CNN
+F 4 "" V 9300 4250 50  0000 R CNN "Placement"
+	1    9300 4200
+	0    1    -1   0
+$EndComp
+$Comp
+L Isolator:LTV-357T U?
+U 1 1 618FB8D7
+P 8600 4300
+AR Path="/60135668/618FB8D7" Ref="U?"  Part="1"
+AR Path="/6044FE50/618FB8D7" Ref="U?"  Part="1"
+AR Path="/5FFC49DA/618FB8D7" Ref="U202"  Part="1"
+F 0 "U202" H 8600 4625 50  0000 C CNN
+F 1 "LTV-357T" H 8600 4534 50  0000 C CNN
+F 2 "Package_SO:SO-4_4.4x3.6mm_P2.54mm" H 8400 4100 50  0001 L CIN
+F 3 "https://www.buerklin.com/medias/sys_master/download/download/h91/ha0/8892020588574.pdf" H 8600 4300 50  0001 L CNN
+F 4 "Lite-On LTV-357T" H 8600 4300 50  0001 C CNN "Bauteil"
+	1    8600 4300
+	-1   0    0    -1
+$EndComp
+$Comp
+L power:+3.3V #PWR?
+U 1 1 618FB8E1
+P 8100 3600
+AR Path="/60135668/618FB8E1" Ref="#PWR?"  Part="1"
+AR Path="/6044FE50/618FB8E1" Ref="#PWR?"  Part="1"
+AR Path="/5FFC49DA/618FB8E1" Ref="#PWR0204"  Part="1"
+F 0 "#PWR0204" H 8100 3450 50  0001 C CNN
+F 1 "+3.3V" H 8115 3773 50  0000 C CNN
+F 2 "" H 8100 3600 50  0001 C CNN
+F 3 "" H 8100 3600 50  0001 C CNN
+	1    8100 3600
+	-1   0    0    -1
+$EndComp
+$Comp
+L power:GND #PWR?
+U 1 1 618FB8E7
+P 8250 4650
+AR Path="/60135668/618FB8E7" Ref="#PWR?"  Part="1"
+AR Path="/6044FE50/618FB8E7" Ref="#PWR?"  Part="1"
+AR Path="/5FFC49DA/618FB8E7" Ref="#PWR0207"  Part="1"
+F 0 "#PWR0207" H 8250 4400 50  0001 C CNN
+F 1 "GND" H 8255 4477 50  0000 C CNN
+F 2 "" H 8250 4650 50  0001 C CNN
+F 3 "" H 8250 4650 50  0001 C CNN
+	1    8250 4650
+	-1   0    0    -1
+$EndComp
+$Comp
+L Device:R R203
+U 1 1 618FB8EE
+P 8100 3750
+AR Path="/5FFC49DA/618FB8EE" Ref="R203"  Part="1"
+AR Path="/6002EA57/618FB8EE" Ref="R?"  Part="1"
+AR Path="/60135668/618FB8EE" Ref="R?"  Part="1"
+AR Path="/6044FE50/618FB8EE" Ref="R?"  Part="1"
+F 0 "R203" H 8030 3659 50  0000 R CNN
+F 1 "4k7" H 8030 3750 50  0000 R CNN
+F 2 "Resistor_SMD:R_0603_1608Metric" V 8030 3750 50  0001 C CNN
+F 3 "~" H 8100 3750 50  0001 C CNN
+F 4 "" V 8100 3800 50  0000 R CNN "Placement"
+	1    8100 3750
+	-1   0    0    -1
+$EndComp
+Wire Wire Line
+	8100 3900 8100 4200
+Wire Wire Line
+	8300 4400 8250 4400
+Wire Wire Line
+	8250 4400 8250 4650
+Wire Wire Line
+	8300 4200 8100 4200
+Wire Wire Line
+	7550 4650 7550 4600
+$Comp
+L power:GND #PWR?
+U 1 1 618FB8F9
+P 7550 4650
+AR Path="/60135668/618FB8F9" Ref="#PWR?"  Part="1"
+AR Path="/6044FE50/618FB8F9" Ref="#PWR?"  Part="1"
+AR Path="/5FFC49DA/618FB8F9" Ref="#PWR0206"  Part="1"
+F 0 "#PWR0206" H 7550 4400 50  0001 C CNN
+F 1 "GND" H 7555 4477 50  0000 C CNN
+F 2 "" H 7550 4650 50  0001 C CNN
+F 3 "" H 7550 4650 50  0001 C CNN
+	1    7550 4650
+	-1   0    0    -1
+$EndComp
+Wire Wire Line
+	7550 4300 7550 4200
+$Comp
+L Device:C C?
+U 1 1 618FB902
+P 7550 4450
+AR Path="/6002EA57/618FB902" Ref="C?"  Part="1"
+AR Path="/6008B538/618FB902" Ref="C?"  Part="1"
+AR Path="/60135668/618FB902" Ref="C?"  Part="1"
+AR Path="/6044FE50/618FB902" Ref="C?"  Part="1"
+AR Path="/5FFC49DA/618FB902" Ref="C201"  Part="1"
+F 0 "C201" H 7665 4541 50  0000 L CNN
+F 1 "100n" H 7665 4450 50  0000 L CNN
+F 2 "Capacitor_SMD:C_0603_1608Metric" H 7588 4300 50  0001 C CNN
+F 3 "~" H 7550 4450 50  0001 C CNN
+F 4 "" H 7665 4359 50  0000 L CNN "Placement"
+F 5 "WE 885382206004" H 7550 4450 50  0001 C CNN "Bauteil"
+	1    7550 4450
+	1    0    0    1
+$EndComp
+$Comp
+L Device:R R204
+U 1 1 618FB909
+P 7850 4200
+AR Path="/5FFC49DA/618FB909" Ref="R204"  Part="1"
+AR Path="/6002EA57/618FB909" Ref="R?"  Part="1"
+AR Path="/60135668/618FB909" Ref="R?"  Part="1"
+AR Path="/6044FE50/618FB909" Ref="R?"  Part="1"
+F 0 "R204" H 7780 4109 50  0000 R CNN
+F 1 "10k" H 7780 4200 50  0000 R CNN
+F 2 "Resistor_SMD:R_0603_1608Metric" V 7780 4200 50  0001 C CNN
+F 3 "~" H 7850 4200 50  0001 C CNN
+F 4 "" V 7850 4250 50  0000 R CNN "Placement"
+	1    7850 4200
+	0    -1   1    0
+$EndComp
+Wire Wire Line
+	8100 4200 8000 4200
+Connection ~ 8100 4200
+Wire Wire Line
+	7700 4200 7550 4200
+Connection ~ 7550 4200
+Wire Wire Line
+	3300 4200 7550 4200
+$Comp
+L power:Earth #PWR?
+U 1 1 61921B5A
+P 8900 4650
+AR Path="/6002EA57/61921B5A" Ref="#PWR?"  Part="1"
+AR Path="/5FFC49DA/61921B5A" Ref="#PWR0208"  Part="1"
+F 0 "#PWR0208" H 8900 4400 50  0001 C CNN
+F 1 "Earth" H 8900 4500 50  0001 C CNN
+F 2 "" H 8900 4650 50  0001 C CNN
+F 3 "~" H 8900 4650 50  0001 C CNN
+	1    8900 4650
+	1    0    0    -1
+$EndComp
+Wire Wire Line
+	8900 4400 8900 4650
+Wire Wire Line
+	8900 4200 9150 4200
+Text GLabel 10100 4200 2    50   Input ~ 0
 TA_Aktiv
-Wire Wire Line
-	3300 4200 5550 4200
+$Comp
+L Device:D D?
+U 1 1 6119AAD9
+P 9750 4200
+AR Path="/6008B538/6119AAD9" Ref="D?"  Part="1"
+AR Path="/60135668/6119AAD9" Ref="D?"  Part="1"
+AR Path="/5FFC49DA/6119AAD9" Ref="D202"  Part="1"
+F 0 "D202" H 9750 3983 50  0000 C CNN
+F 1 "1N4148" H 9750 4074 50  0000 C CNN
+F 2 "Diode_SMD:D_SOD-323F" H 9750 4200 50  0001 C CNN
+F 3 "~" H 9750 4200 50  0001 C CNN
+F 4 "ON 1N4148WS" H 9750 4200 50  0001 C CNN "Bauteil"
+	1    9750 4200
+	1    0    0    -1
+$EndComp
+Wire Wire Line
+	9450 4200 9600 4200
+Wire Wire Line
+	9900 4200 10100 4200
 $EndSCHEMATC
