File: cad/pcb/saba-fernbedienung/rev2-a/2-steckverbinder.sch (KiCad schematic (older format))
At the start: 29 parts, among them J301 Conn_01x04, J302 Conn_01x04, J303 Micro_SD_Card, J304 Conn_01x04, J305 AudioJack3, J306 Conn_01x02, J307 Conn_01x04, J308 Conn_01x01, J309 Conn_01x01, J310 Conn_01x01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

Commit message: ToDo-s bearbeitet
Parts:
- removed J312: Conn_01x08, Connector_PinHeader_2.54mm:PinHeader_2x04_P2.54mm_Vertical, symbol Connector_Generic:Conn_01x08
- removed R301, R302: 1k, Resistor_SMD:R_0603_1608Metric, symbol Device:R
- removed R303: 0, Resistor_SMD:R_0603_1608Metric, symbol Device:R
Connections:
- net Audio_Links: now also D301.2 (A2), J305.T, J310.1 (Pin_1)
- net Audio_Rechts: now also D301.1 (A1), J305.R, J309.1 (Pin_1)
- net GND: no longer D301.3 (common), J305.T, J308.1 (Pin_1)
- net TA_Aktiv: now reaches J311.1 (Pin_1)
- new net Audio_GND: D301.3 (common), J305.S, J308.1 (Pin_1)
- no-connect marks 12 -> 11
Other:
- note removed: "Optional: Stereo - 2x 0R"
- note removed: "TFT (optional)"
- moved on the sheet: C304, D301, J305, J308, J309, J310, R305, U301

Commit message: Change: Bauteilbezeichner
Parts:
- renumbered J313 to J312, R304 to R301, R305 to R302, R306 to R303, R307 to R304, R308 to R305
Changed lines of the file:
@@
 Anschlussstecker Radio
 $Comp
-L Connector:USB_C_Receptacle_USB2.0 J313
+L Connector:USB_C_Receptacle_USB2.0 J312
 U 1 1 6005055F
 P 1850 5250
-F 0 "J313" H 1957 6207 50  0000 C CNN
+F 0 "J312" H 1957 6207 50  0000 C CNN
 F 1 "USB_C_Receptacle_USB2.0" H 1957 6116 50  0000 C CNN
 F 2 "Connector_USB:USB_C_Receptacle_HRO_TYPE-C-31-M-12" H 2000 5250 50  0001 C CNN
@@
 Spannungsversorgung USB (optional)
 $Comp
-L power:GND #PWR0319
+L power:GND #PWR0316
 U 1 1 60063A29
 P 1850 6700
-F 0 "#PWR0319" H 1850 6450 50  0001 C CNN
+F 0 "#PWR0316" H 1850 6450 50  0001 C CNN
 F 1 "GND" H 1855 6527 50  0000 C CNN
 F 2 "" H 1850 6700 50  0001 C CNN
@@
 	2450 4950 2700 4950
 $Comp
-L power:GND #PWR0315
+L power:GND #PWR0312
 U 1 1 6006013B
 P 3150 5550
-F 0 "#PWR0315" H 3150 5300 50  0001 C CNN
+F 0 "#PWR0312" H 3150 5300 50  0001 C CNN
 F 1 "GND" H 3155 5377 50  0000 C CNN
 F 2 "" H 3150 5550 50  0001 C CNN
@@
 $EndComp
 $Comp
-L power:GND #PWR0314
+L power:GND #PWR0311
 U 1 1 6005FCD0
 P 2700 5550
-F 0 "#PWR0314" H 2700 5300 50  0001 C CNN
+F 0 "#PWR0311" H 2700 5300 50  0001 C CNN
 F 1 "GND" H 2705 5377 50  0000 C CNN
 F 2 "" H 2700 5550 50  0001 C CNN
@@
 P 3150 5300
 AR Path="/5FFC49DA/6005BEE2" Ref="R?"  Part="1"
-AR Path="/6002EA57/6005BEE2" Ref="R307"  Part="1"
-F 0 "R307" H 3220 5391 50  0000 L CNN
+AR Path="/6002EA57/6005BEE2" Ref="R304"  Part="1"
+F 0 "R304" H 3220 5391 50  0000 L CNN
 F 1 "5k1" H 3220 5300 50  0000 L CNN
 F 2 "Resistor_SMD:R_0603_1608Metric" V 3080 5300 50  0001 C CNN
@@
 P 2700 5300
 AR Path="/5FFC49DA/6005B9D4" Ref="R?"  Part="1"
-AR Path="/6002EA57/6005B9D4" Ref="R306"  Part="1"
-F 0 "R306" H 2630 5209 50  0000 R CNN
+AR Path="/6002EA57/6005B9D4" Ref="R303"  Part="1"
+F 0 "R303" H 2630 5209 50  0000 R CNN
 F 1 "5k1" H 2630 5300 50  0000 R CNN
 F 2 "Resistor_SMD:R_0603_1608Metric" V 2630 5300 50  0001 C CNN
@@
 	2450 4650 3550 4650
 $Comp
-L power:GND #PWR0316
+L power:GND #PWR0313
 U 1 1 600712E7
 P 3550 5550
-F 0 "#PWR0316" H 3550 5300 50  0001 C CNN
+F 0 "#PWR0313" H 3550 5300 50  0001 C CNN
 F 1 "GND" H 3555 5377 50  0000 C CNN
 F 2 "" H 3550 5550 50  0001 C CNN
@@
 $EndComp
 $Comp
-L power:GND #PWR0317
+L power:GND #PWR0314
 U 1 1 6007D5DC
 P 4100 5550
-F 0 "#PWR0317" H 4100 5300 50  0001 C CNN
+F 0 "#PWR0314" H 4100 5300 50  0001 C CNN
 F 1 "GND" H 4105 5377 50  0000 C CNN
 F 2 "" H 4100 5550 50  0001 C CNN
@@
 	4100 4650 4500 4650
 $Comp
-L power:+5V #PWR0309
+L power:+5V #PWR0308
 U 1 1 60082BAA
 P 5100 4600
-F 0 "#PWR0309" H 5100 4450 50  0001 C CNN
+F 0 "#PWR0308" H 5100 4450 50  0001 C CNN
 F 1 "+5V" H 5115 4773 50  0000 C CNN
 F 2 "" H 5100 4600 50  0001 C CNN
@@
 P 1550 6400
 AR Path="/5FFC49DA/5FFDECFB" Ref="R?"  Part="1"
-AR Path="/6002EA57/5FFDECFB" Ref="R308"  Part="1"
-F 0 "R308" H 1480 6309 50  0000 R CNN
+AR Path="/6002EA57/5FFDECFB" Ref="R305"  Part="1"
+F 0 "R305" H 1480 6309 50  0000 R CNN
 F 1 "1M" H 1480 6400 50  0000 R CNN
 F 2 "Resistor_SMD:R_0603_1608Metric" V 1480 6400 50  0001 C CNN
@@
 P 6600 3000
 AR Path="/5FFC49DA/5FFE4E96" Ref="R?"  Part="1"
-AR Path="/6002EA57/5FFE4E96" Ref="R304"  Part="1"
-F 0 "R304" H 6530 2909 50  0000 R CNN
+AR Path="/6002EA57/5FFE4E96" Ref="R301"  Part="1"
+F 0 "R301" H 6530 2909 50  0000 R CNN
 F 1 "1M" H 6530 3000 50  0000 R CNN
 F 2 "Resistor_SMD:R_0603_1608Metric" V 6530 3000 50  0001 C CNN
@@
 $EndComp
 $Comp
-L power:GND #PWR0312
+L power:GND #PWR0310
 U 1 1 6001F94B
 P 6750 5200
-F 0 "#PWR0312" H 6750 4950 50  0001 C CNN
+F 0 "#PWR0310" H 6750 4950 50  0001 C CNN
 F 1 "GND" H 6755 5027 50  0000 C CNN
 F 2 "" H 6750 5200 50  0001 C CNN
@@
 	8100 4550 8100 4650
 $Comp
-L power:+3.3V #PWR0308
+L power:+3.3V #PWR0307
 U 1 1 60021397
 P 8100 4550
-F 0 "#PWR0308" H 8100 4400 50  0001 C CNN
+F 0 "#PWR0307" H 8100 4400 50  0001 C CNN
 F 1 "+3.3V" H 8115 4723 50  0000 C CNN
 F 2 "" H 8100 4550 50  0001 C CNN
@@
 $EndComp
 $Comp
-L power:GND #PWR0311
+L power:GND #PWR0309
 U 1 1 60020161
 P 7400 5150
-F 0 "#PWR0311" H 7400 4900 50  0001 C CNN
+F 0 "#PWR0309" H 7400 4900 50  0001 C CNN
 F 1 "GND" H 7405 4977 50  0000 C CNN
 F 2 "" H 7400 5150 50  0001 C CNN
@@
 P 7850 4650
 AR Path="/5FFC49DA/6001BDE1" Ref="R?"  Part="1"
-AR Path="/6002EA57/6001BDE1" Ref="R305"  Part="1"
-F 0 "R305" H 7780 4559 50  0000 R CNN
+AR Path="/6002EA57/6001BDE1" Ref="R302"  Part="1"
+F 0 "R302" H 7780 4559 50  0000 R CNN
 F 1 "100" H 7780 4650 50  0000 R CNN
 F 2 "Resistor_SMD:R_0603_1608Metric" V 7780 4650 50  0001 C CNN
@@
 $EndComp
 $Comp
-L power:GND #PWR0101
+L power:GND #PWR0306
 U 1 1 6003FF39
 P 6600 3250
-F 0 "#PWR0101" H 6600 3000 50  0001 C CNN
+F 0 "#PWR0306" H 6600 3000 50  0001 C CNN
 F 1 "GND" H 6605 3077 50  0000 C CNN
 F 2 "" H 6600 3250 50  0001 C CNN
@@
 $EndComp
 $Comp
-L power:GND #PWR0103
+L power:GND #PWR0315
 U 1 1 60040E02
 P 1550 6700
-F 0 "#PWR0103" H 1550 6450 50  0001 C CNN
+F 0 "#PWR0315" H 1550 6450 50  0001 C CNN
 F 1 "GND" H 1555 6527 50  0000 C CNN
 F 2 "" H 1550 6700 50  0001 C CNN

Commit message: Sicherung
Parts:
- removed D301: 5V, Package_TO_SOT_SMD:SOT-323_SC-70, symbol Device:D_TVS_x2_AAC
Changed lines of the file:
@@
 	1    0    0    -1
 $EndComp
-Wire Wire Line
-	4850 3450 4850 3500
 NoConn ~ 2450 5150
 NoConn ~ 2450 5250
@@
 Audio_GND
 Wire Wire Line
-	4500 2300 4700 2300
-Wire Wire Line
-	4500 2200 4850 2200
-Wire Wire Line
-	4850 2200 4850 2750
-Wire Wire Line
-	4500 2100 5000 2100
-Wire Wire Line
-	5000 3500 4850 3500
-$Comp
-L Device:D_TVS_x2_AAC D301
-U 1 1 609A1EE5
-P 4850 3100
-F 0 "D301" V 4950 2750 50  0000 L CNN
-F 1 "5V" V 5050 2800 50  0000 L CNN
-F 2 "Package_TO_SOT_SMD:SOT-323_SC-70" H 4700 3100 50  0001 C CNN
-F 3 "https://www.diodes.com/assets/Datasheets/D5V0L2B3W.pdf" H 4700 3100 50  0001 C CNN
-F 4 "Diodes D5V0L2B3W" V 4850 3100 50  0001 C CNN "Bauteil"
-	1    4850 3100
-	0    1    1    0
-$EndComp
-Wire Wire Line
-	4700 2300 5100 2300
-Wire Wire Line
 	5500 2300 5500 2650
-Connection ~ 4700 2300
-Wire Wire Line
-	4850 2200 5250 2200
 Wire Wire Line
 	5650 2200 5650 2650
-Connection ~ 4850 2200
-Wire Wire Line
-	5000 2100 5400 2100
 Wire Wire Line
 	5800 2100 5800 2650
-Connection ~ 5000 2100
-Wire Wire Line
-	5000 2100 5000 3500
 Text GLabel 5400 1750 1    50   Input ~ 0
 Audio_Links
@@
 	5400 2100 5800 2100
 Wire Wire Line
-	4700 2300 4700 3100
-Wire Wire Line
 	2250 3200 1850 3200
 Text GLabel 2250 3200 2    50   Input ~ 0
 TA_Aktiv
+Wire Wire Line
+	4500 2300 5100 2300
+Wire Wire Line
+	4500 2200 5250 2200
+Wire Wire Line
+	4500 2100 5400 2100
 $EndSCHEMATC

Commit message: Update NP, Fix ToDo-s
Parts:
- C304, R302, U301: Placement (none) -> NP
Changed lines of the file:
@@
 Sheet 3 7
 Title "Fernbedienung - Webradio SABA 6-3D"
-Date "2021-08-14"
+Date "2022-06-05"
 Rev "2-A"
 Comp "Martin Wagner DL2WAG"
@@
 F 3 "http://www.vishay.com/docs/82492/tsop312.pdf" H 6900 5150 50  0001 C CNN
 F 4 "Vishay TSOP31238" H 6250 4850 50  0001 C CNN "Bauteil"
+F 5 "NP" H 6250 4850 50  0000 C CNN "Placement"
 	1    6250 4850
 	1    0    0    -1
@@
 F 2 "Capacitor_SMD:C_0603_1608Metric" H 7438 4750 50  0001 C CNN
 F 3 "~" H 7400 4900 50  0001 C CNN
-F 4 "" H 7515 4809 50  0000 L CNN "Placement"
+F 4 "NP" H 7515 4809 50  0000 L CNN "Placement"
 F 5 "WE 885382206004" H 7400 4900 50  0001 C CNN "Bauteil"
 	1    7400 4900
@@
 F 2 "Resistor_SMD:R_0603_1608Metric" V 7780 4650 50  0001 C CNN
 F 3 "~" H 7850 4650 50  0001 C CNN
-F 4 "" V 7850 4700 50  0000 R CNN "Placement"
+F 4 "NP" V 7850 4700 50  0000 R CNN "Placement"
 	1    7850 4650
 	0    -1   -1   0
