File: cad/pcb/saba-fernbedienung/rev2-a/3-spannungsversorgung.sch (KiCad schematic (older format))
At the start: 32 parts, among them U401 TEC2-0911, U402 1117 1.8V, U403 1117 3.3V

Commit message: ToDo-s bearbeitet
Parts:
- removed C401: 150p, Capacitor_SMD:C_0603_1608Metric, symbol Device:C
- removed C404: 10u, Capacitor_SMD:C_1206_3216Metric, symbol Device:C
- removed C406: 100n, Capacitor_SMD:C_0603_1608Metric, symbol Device:C
- removed C409: 220p, Capacitor_SMD:C_0603_1608Metric, symbol Device:C
- removed L401: 4,7u, local:WE-LQ, symbol Device:L
- removed U401: TEC2-0911, local:Converter_DCDC_TRACO_TEC2_xxxx_THT, symbol local:TEC2-0911
- added C?: 10u, Capacitor_SMD:C_1206_3216Metric, symbol Device:C
- added D?: B140-E3, Diode_SMD:D_SMA, symbol Diode:B140-E3
- added U?: 1117 5.0V, Package_TO_SOT_SMD:TO-252-3_TabPin2, symbol Regulator_Linear:AP1117-18
Connections:
- net +3.3VA: now also D?.2 (A)
- net +5V: now also C?.1, U?.2 (VO)
- net GND: now also C402.2, C403.2, C405.2, D403.2 (A), D404.2 (A), C?.2, U?.1 (GND)
- net at C402.1, C403.1, D401.1 (K)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: now also C405.1, U?.3 (VI)
- new net +3V3: D?.1 (K)
- no-connect marks 1 -> 0
Other:
- note added: "3V3 darf nicht in der Luft \nhängen wenn ESP32 nicht \ngesteckt ist"
- note added: "Spannungsversorgung 5V"
- note removed: "Nach "TEC 2 Series EMI Consideration, Class B""
- note removed: "Spannungsversorgung 5V mit Trennung GND"
- moved on the sheet: C405, C407

Commit message: Change: Bauteilbezeichner
Parts:
- gave numbers to parts that had none: 3
- renumbered C402 to C401, C403 to C402, C405 to C403, C407 to C405, C408 to C406, C410 to C407, C411 to C408, C412 to C409, C413 to C410, C414 to C411, C415 to C412, C416 to C413, C417 to C414, C418 to C415, C419 to C416, D406 to D407, L402 to L401
Changed lines of the file:
@@
 P 3000 1950
 AR Path="/6002EA57/600BAEBF" Ref="C?"  Part="1"
-AR Path="/6008B538/600BAEBF" Ref="C402"  Part="1"
-F 0 "C402" H 3115 2041 50  0000 L CNN
+AR Path="/6008B538/600BAEBF" Ref="C401"  Part="1"
+F 0 "C401" H 3115 2041 50  0000 L CNN
 F 1 "100n" H 3115 1950 50  0000 L CNN
 F 2 "Capacitor_SMD:C_0603_1608Metric" H 3038 1800 50  0001 C CNN
@@
 P 1650 2000
 AR Path="/6002EA57/600C5AD1" Ref="C?"  Part="1"
-AR Path="/6008B538/600C5AD1" Ref="C408"  Part="1"
-F 0 "C408" H 1765 2091 50  0000 L CNN
+AR Path="/6008B538/600C5AD1" Ref="C406"  Part="1"
+F 0 "C406" H 1765 2091 50  0000 L CNN
 F 1 "100n" H 1765 2000 50  0000 L CNN
 F 2 "Capacitor_SMD:C_0603_1608Metric" H 1688 1850 50  0001 C CNN
@@
 P 4500 1950
 AR Path="/6002EA57/600C92CE" Ref="C?"  Part="1"
-AR Path="/6008B538/600C92CE" Ref="C405"  Part="1"
-F 0 "C405" H 4615 2041 50  0000 L CNN
+AR Path="/6008B538/600C92CE" Ref="C403"  Part="1"
+F 0 "C403" H 4615 2041 50  0000 L CNN
 F 1 "10u" H 4615 1950 50  0000 L CNN
 F 2 "Capacitor_SMD:C_1206_3216Metric" H 4538 1800 50  0001 C CNN
@@
 	3000 2700 3450 2700
 $Comp
-L Device:CP C407
+L Device:CP C405
 U 1 1 600DE083
 P 6750 1950
-F 0 "C407" H 6868 2041 50  0000 L CNN
+F 0 "C405" H 6868 2041 50  0000 L CNN
 F 1 "220u" H 6868 1950 50  0000 L CNN
 F 2 "local:CP_Radial_D10.0mm_P5.00mm_liegend" H 6788 1800 50  0001 C CNN
@@
 	3450 1800 3450 1300
 $Comp
-L Device:CP C403
+L Device:CP C402
 U 1 1 600BF78B
 P 3450 1950
-F 0 "C403" H 3568 2041 50  0000 L CNN
+F 0 "C402" H 3568 2041 50  0000 L CNN
 F 1 "1000u" H 3568 1950 50  0000 L CNN
 F 2 "Capacitor_THT:CP_Radial_D10.0mm_P5.00mm" H 3488 1800 50  0001 C CNN
@@
 $EndComp
 $Comp
-L Device:D D406
+L Device:D D407
 U 1 1 60100DBC
 P 2050 5400
-F 0 "D406" H 2050 5617 50  0000 C CNN
+F 0 "D407" H 2050 5617 50  0000 C CNN
 F 1 "1N4007" H 2050 5526 50  0000 C CNN
 F 2 "Diode_SMD:D_SMA" H 2050 5400 50  0001 C CNN
@@
 $EndComp
 $Comp
-L Device:CP C410
+L Device:CP C407
 U 1 1 60101A51
 P 2600 4350
-F 0 "C410" H 2718 4441 50  0000 L CNN
+F 0 "C407" H 2718 4441 50  0000 L CNN
 F 1 "220u" H 2718 4350 50  0000 L CNN
 F 2 "Capacitor_THT:CP_Radial_D10.0mm_P5.00mm" H 2638 4200 50  0001 C CNN
@@
 P 3100 4350
 AR Path="/6002EA57/60102210" Ref="C?"  Part="1"
-AR Path="/6008B538/60102210" Ref="C411"  Part="1"
-F 0 "C411" H 3215 4441 50  0000 L CNN
+AR Path="/6008B538/60102210" Ref="C408"  Part="1"
+F 0 "C408" H 3215 4441 50  0000 L CNN
 F 1 "100n" H 3215 4350 50  0000 L CNN
 F 2 "Capacitor_SMD:C_0603_1608Metric" H 3138 4200 50  0001 C CNN
@@
 P 3100 5050
 AR Path="/6002EA57/60103644" Ref="C?"  Part="1"
-AR Path="/6008B538/60103644" Ref="C419"  Part="1"
-F 0 "C419" H 3215 5141 50  0000 L CNN
+AR Path="/6008B538/60103644" Ref="C416"  Part="1"
+F 0 "C416" H 3215 5141 50  0000 L CNN
 F 1 "100n" H 3215 5050 50  0000 L CNN
 F 2 "Capacitor_SMD:C_0603_1608Metric" H 3138 4900 50  0001 C CNN
@@
 	3100 4700 3100 4900
 $Comp
-L Device:CP C418
+L Device:CP C415
 U 1 1 6010F424
 P 2600 5050
-F 0 "C418" H 2718 5141 50  0000 L CNN
+F 0 "C415" H 2718 5141 50  0000 L CNN
 F 1 "220u" H 2718 5050 50  0000 L CNN
 F 2 "Capacitor_THT:CP_Radial_D10.0mm_P5.00mm" H 2638 4900 50  0001 C CNN
@@
 	2600 4700 2600 4900
 $Comp
-L power:-24V #PWR0415
+L power:-24V #PWR0416
 U 1 1 601188A7
 P 3300 5500
-F 0 "#PWR0415" H 3300 5600 50  0001 C CNN
+F 0 "#PWR0416" H 3300 5600 50  0001 C CNN
 F 1 "-24V" H 3315 5673 50  0000 C CNN
 F 2 "" H 3300 5500 50  0001 C CNN
@@
 P 4450 5050
 AR Path="/6002EA57/6044C3D0" Ref="#PWR?"  Part="1"
-AR Path="/6008B538/6044C3D0" Ref="#PWR0409"  Part="1"
-F 0 "#PWR0409" H 4450 4800 50  0001 C CNN
+AR Path="/6008B538/6044C3D0" Ref="#PWR0410"  Part="1"
+F 0 "#PWR0410" H 4450 4800 50  0001 C CNN
 F 1 "GND" H 4455 4877 50  0000 C CNN
 F 2 "" H 4450 5050 50  0001 C CNN
@@
 P 5000 5050
 AR Path="/6002EA57/6044CA24" Ref="#PWR?"  Part="1"
-AR Path="/6008B538/6044CA24" Ref="#PWR0410"  Part="1"
-F 0 "#PWR0410" H 5000 4800 50  0001 C CNN
+AR Path="/6008B538/6044CA24" Ref="#PWR0411"  Part="1"
+F 0 "#PWR0411" H 5000 4800 50  0001 C CNN
 F 1 "GND" H 5005 4877 50  0000 C CNN
 F 2 "" H 5000 5050 50  0001 C CNN
@@
 P 5500 5050
 AR Path="/6002EA57/6044CEF7" Ref="#PWR?"  Part="1"
-AR Path="/6008B538/6044CEF7" Ref="#PWR0411"  Part="1"
-F 0 "#PWR0411" H 5500 4800 50  0001 C CNN
+AR Path="/6008B538/6044CEF7" Ref="#PWR0412"  Part="1"
+F 0 "#PWR0412" H 5500 4800 50  0001 C CNN
 F 1 "GND" H 5505 4877 50  0000 C CNN
 F 2 "" H 5500 5050 50  0001 C CNN
@@
 P 6850 5050
 AR Path="/6002EA57/6044D301" Ref="#PWR?"  Part="1"
-AR Path="/6008B538/6044D301" Ref="#PWR0412"  Part="1"
-F 0 "#PWR0412" H 6850 4800 50  0001 C CNN
+AR Path="/6008B538/6044D301" Ref="#PWR0413"  Part="1"
+F 0 "#PWR0413" H 6850 4800 50  0001 C CNN
 F 1 "GND" H 6855 4877 50  0000 C CNN
 F 2 "" H 6850 5050 50  0001 C CNN
@@
 P 7350 5050
 AR Path="/6002EA57/6044D957" Ref="#PWR?"  Part="1"
-AR Path="/6008B538/6044D957" Ref="#PWR0413"  Part="1"
-F 0 "#PWR0413" H 7350 4800 50  0001 C CNN
+AR Path="/6008B538/6044D957" Ref="#PWR0414"  Part="1"
+F 0 "#PWR0414" H 7350 4800 50  0001 C CNN
 F 1 "GND" H 7355 4877 50  0000 C CNN
 F 2 "" H 7350 5050 50  0001 C CNN
@@
 P 7800 5050
 AR Path="/6002EA57/6044DE01" Ref="#PWR?"  Part="1"
-AR Path="/6008B538/6044DE01" Ref="#PWR0414"  Part="1"
-F 0 "#PWR0414" H 7800 4800 50  0001 C CNN
+AR Path="/6008B538/6044DE01" Ref="#PWR0415"  Part="1"
+F 0 "#PWR0415" H 7800 4800 50  0001 C CNN
 F 1 "GND" H 7805 4877 50  0000 C CNN
 F 2 "" H 7800 5050 50  0001 C CNN
@@
 Spannungsversorgung Audio Codec/DAC\n
 $Comp
-L Device:L L402
+L Device:L L401
 U 1 1 60483E20
 P 6650 4400
-F 0 "L402" V 6840 4400 50  0000 C CNN
+F 0 "L401" V 6840 4400 50  0000 C CNN
 F 1 "4,7u" V 6749 4400 50  0000 C CNN
 F 2 "local:WE-LQ" H 6650 4400 50  0001 C CNN
@@
 P 4450 4800
 AR Path="/6002EA57/6003B8AE" Ref="C?"  Part="1"
-AR Path="/6008B538/6003B8AE" Ref="C412"  Part="1"
-F 0 "C412" H 4565 4891 50  0000 L CNN
+AR Path="/6008B538/6003B8AE" Ref="C409"  Part="1"
+F 0 "C409" H 4565 4891 50  0000 L CNN
 F 1 "10u" H 4565 4800 50  0000 L CNN
 F 2 "Capacitor_SMD:C_1206_3216Metric" H 4488 4650 50  0001 C CNN
@@
 P 5500 4800
 AR Path="/6002EA57/6003C248" Ref="C?"  Part="1"
-AR Path="/6008B538/6003C248" Ref="C413"  Part="1"
-F 0 "C413" H 5615 4891 50  0000 L CNN
+AR Path="/6008B538/6003C248" Ref="C410"  Part="1"
+F 0 "C410" H 5615 4891 50  0000 L CNN
 F 1 "10u" H 5615 4800 50  0000 L CNN
 F 2 "Capacitor_SMD:C_1206_3216Metric" H 5538 4650 50  0001 C CNN
@@
 P 5850 4800
 AR Path="/6002EA57/6003C938" Ref="C?"  Part="1"
-AR Path="/6008B538/6003C938" Ref="C414"  Part="1"
-F 0 "C414" H 5965 4891 50  0000 L CNN
+AR Path="/6008B538/6003C938" Ref="C411"  Part="1"
+F 0 "C411" H 5965 4891 50  0000 L CNN
 F 1 "10u" H 5965 4800 50  0000 L CNN
 F 2 "Capacitor_SMD:C_1206_3216Metric" H 5888 4650 50  0001 C CNN
@@
 P 6850 4800
 AR Path="/6002EA57/6003CCE9" Ref="C?"  Part="1"
-AR Path="/6008B538/6003CCE9" Ref="C415"  Part="1"
-F 0 "C415" H 6965 4891 50  0000 L CNN
+AR Path="/6008B538/6003CCE9" Ref="C412"  Part="1"
+F 0 "C412" H 6965 4891 50  0000 L CNN
 F 1 "10u" H 6965 4800 50  0000 L CNN
 F 2 "Capacitor_SMD:C_1206_3216Metric" H 6888 4650 50  0001 C CNN
@@
 P 7800 4800
 AR Path="/6002EA57/6003D22E" Ref="C?"  Part="1"
-AR Path="/6008B538/6003D22E" Ref="C416"  Part="1"
-F 0 "C416" H 7915 4891 50  0000 L CNN
+AR Path="/6008B538/6003D22E" Ref="C413"  Part="1"
+F 0 "C413" H 7915 4891 50  0000 L CNN
 F 1 "10u" H 7915 4800 50  0000 L CNN
 F 2 "Capacitor_SMD:C_1206_3216Metric" H 7838 4650 50  0001 C CNN
@@
 P 8200 4800
 AR Path="/6002EA57/6003D8C4" Ref="C?"  Part="1"
-AR Path="/6008B538/6003D8C4" Ref="C417"  Part="1"
-F 0 "C417" H 8315 4891 50  0000 L CNN
+AR Path="/6008B538/6003D8C4" Ref="C414"  Part="1"
+F 0 "C414" H 8315 4891 50  0000 L CNN
 F 1 "10u" H 8315 4800 50  0000 L CNN
 F 2 "Capacitor_SMD:C_1206_3216Metric" H 8238 4650 50  0001 C CNN
@@
 P 9350 4050
 AR Path="/5FFC49DA/611C7361" Ref="#PWR?"  Part="1"
-AR Path="/6008B538/611C7361" Ref="#PWR?"  Part="1"
-F 0 "#PWR?" H 9350 3900 50  0001 C CNN
+AR Path="/6008B538/611C7361" Ref="#PWR0409"  Part="1"
+F 0 "#PWR0409" H 9350 3900 50  0001 C CNN
 F 1 "+3V3" H 9365 4223 50  0000 C CNN
 F 2 "" H 9350 4050 50  0001 C CNN
@@
 P 9000 4400
 AR Path="/6002EA57/611CB2E1" Ref="D?"  Part="1"
-AR Path="/6008B538/611CB2E1" Ref="D?"  Part="1"
-F 0 "D?" H 9000 4150 50  0000 C CNN
+AR Path="/6008B538/611CB2E1" Ref="D406"  Part="1"
+F 0 "D406" H 9000 4150 50  0000 C CNN
 F 1 "B140-E3" H 9000 4250 50  0000 C CNN
 F 2 "Diode_SMD:D_SMA" H 9000 4225 50  0001 C CNN
@@
 P 5850 1950
 AR Path="/6002EA57/614C8397" Ref="C?"  Part="1"
-AR Path="/6008B538/614C8397" Ref="C?"  Part="1"
-F 0 "C?" H 5965 2041 50  0000 L CNN
+AR Path="/6008B538/614C8397" Ref="C404"  Part="1"
+F 0 "C404" H 5965 2041 50  0000 L CNN
 F 1 "10u" H 5965 1950 50  0000 L CNN
 F 2 "Capacitor_SMD:C_1206_3216Metric" H 5888 1800 50  0001 C CNN
@@
 	5850 2700 6750 2700
 $Comp
-L Regulator_Linear:AP1117-18 U?
+L Regulator_Linear:AP1117-18 U401
 U 1 1 6177A88D
 P 5200 1300
-F 0 "U?" H 5200 1542 50  0000 C CNN
+F 0 "U401" H 5200 1542 50  0000 C CNN
 F 1 "1117 5.0V" H 5200 1451 50  0000 C CNN
 F 2 "Package_TO_SOT_SMD:TO-252-3_TabPin2" H 5200 1500 50  0001 C CNN

Commit message: Sicherung
Parts:
- C402: footprint Capacitor_THT:CP_Radial_D10.0mm_P5.00mm -> local:CP_Radial_D10.0mm_P5.00mm_L20.00mm_liegend
- C405: footprint local:CP_Radial_D10.0mm_P5.00mm_liegend -> local:CP_Radial_D10.0mm_P5.00mm_L12.50mm_liegend
Changed lines of the file:
@@
 F 0 "C405" H 6868 2041 50  0000 L CNN
 F 1 "220u" H 6868 1950 50  0000 L CNN
-F 2 "local:CP_Radial_D10.0mm_P5.00mm_liegend" H 6788 1800 50  0001 C CNN
+F 2 "local:CP_Radial_D10.0mm_P5.00mm_L12.50mm_liegend" H 6788 1800 50  0001 C CNN
 F 3 "~" H 6750 1950 50  0001 C CNN
 F 4 "10V" H 6868 1859 50  0000 L CNN "Voltage"
@@
 F 0 "C402" H 3568 2041 50  0000 L CNN
 F 1 "1000u" H 3568 1950 50  0000 L CNN
-F 2 "Capacitor_THT:CP_Radial_D10.0mm_P5.00mm" H 3488 1800 50  0001 C CNN
+F 2 "local:CP_Radial_D10.0mm_P5.00mm_L20.00mm_liegend" H 3488 1800 50  0001 C CNN
 F 3 "~" H 3450 1950 50  0001 C CNN
 F 4 "16V" H 3568 1859 50  0000 L CNN "Voltage"

Commit message: Update NP, Fix ToDo-s
Parts:
- U401: symbol Regulator_Linear:AP1117-18 -> Regulator_Linear:AP1117-50
Changed lines of the file:
@@
 Sheet 4 7
 Title "Fernbedienung - Webradio SABA 6-3D"
-Date "2021-08-14"
+Date "2022-06-05"
 Rev "2-A"
 Comp "Martin Wagner DL2WAG"
@@
 	5850 2700 6750 2700
 $Comp
-L Regulator_Linear:AP1117-18 U401
+L Regulator_Linear:AP1117-50 U401
 U 1 1 6177A88D
 P 5200 1300
