File: cad/pcb/saba-fernbedienung/rev2-a/4-suchlauf-in.sch (KiCad schematic (older format))
At the start: 56 parts, among them U501 ADA4522-2, U502 LM339, U503 LTV-357T, U504 LTV-357T, U505 LTV-357T

Commit message: ToDo-s bearbeitet
Parts:
- R511, R519: value 68k -> 680k
- R512, R515, R529: value 1k -> 10k
- R513, R516, R530: value 1k -> 4k7
- R514: value 27k -> 20k
- R520: value 470k -> 360k
- R521: value 3k3 -> 33k
- R525, R526, R536: value 22k -> 10k
- R528: value 15k -> 150k
- R533: value 18k -> 180k
- R534: value 8k2 -> 82k
Other:
- note added: "18,5V +/-0,5V"
- note removed: "17,5V +/-0,5V"
Changed lines of the file:
@@
 Sheet 5 7
 Title "Fernbedienung - Webradio SABA 6-3D"
-Date "2021-01-16"
-Rev "1-A"
+Date "2021-08-14"
+Rev "2-A"
 Comp "Martin Wagner DL2WAG"
 Comment1 "Lizenz: CERN-OHL-W (OHL v2)"
@@
 AR Path="/60135668/601CB1B5" Ref="R519"  Part="1"
 F 0 "R519" H 2280 4359 50  0000 R CNN
-F 1 "68k" H 2280 4450 50  0000 R CNN
+F 1 "680k" H 2280 4450 50  0000 R CNN
 F 2 "Resistor_SMD:R_0603_1608Metric" V 2280 4450 50  0001 C CNN
 F 3 "~" H 2350 4450 50  0001 C CNN
@@
 AR Path="/60135668/601CBE86" Ref="R511"  Part="1"
 F 0 "R511" H 1630 3409 50  0000 R CNN
-F 1 "68k" H 1630 3500 50  0000 R CNN
+F 1 "680k" H 1630 3500 50  0000 R CNN
 F 2 "Resistor_SMD:R_0603_1608Metric" V 1630 3500 50  0001 C CNN
 F 3 "~" H 1700 3500 50  0001 C CNN
@@
 AR Path="/60135668/601CC823" Ref="R521"  Part="1"
 F 0 "R521" H 1630 4609 50  0000 R CNN
-F 1 "3k3" H 1630 4700 50  0000 R CNN
+F 1 "33k" H 1630 4700 50  0000 R CNN
 F 2 "Resistor_SMD:R_0603_1608Metric" V 1630 4700 50  0001 C CNN
 F 3 "~" H 1700 4700 50  0001 C CNN
@@
 AR Path="/60135668/60207628" Ref="R512"  Part="1"
 F 0 "R512" H 2980 3409 50  0000 R CNN
-F 1 "1k" H 2980 3500 50  0000 R CNN
+F 1 "10k" H 2980 3500 50  0000 R CNN
 F 2 "Resistor_SMD:R_0603_1608Metric" V 2980 3500 50  0001 C CNN
 F 3 "~" H 3050 3500 50  0001 C CNN
@@
 AR Path="/60135668/60218D35" Ref="R513"  Part="1"
 F 0 "R513" H 3880 3409 50  0000 R CNN
-F 1 "1k" H 3880 3500 50  0000 R CNN
+F 1 "4k7" H 3880 3500 50  0000 R CNN
 F 2 "Resistor_SMD:R_0603_1608Metric" V 3880 3500 50  0001 C CNN
 F 3 "~" H 3950 3500 50  0001 C CNN
@@
 AR Path="/60135668/6028371F" Ref="R533"  Part="1"
 F 0 "R533" H 2280 6759 50  0000 R CNN
-F 1 "18k" H 2280 6850 50  0000 R CNN
+F 1 "180k" H 2280 6850 50  0000 R CNN
 F 2 "Resistor_SMD:R_0603_1608Metric" V 2280 6850 50  0001 C CNN
 F 3 "~" H 2350 6850 50  0001 C CNN
@@
 AR Path="/60135668/60283726" Ref="R528"  Part="1"
 F 0 "R528" H 1630 5809 50  0000 R CNN
-F 1 "15k" H 1630 5900 50  0000 R CNN
+F 1 "150k" H 1630 5900 50  0000 R CNN
 F 2 "Resistor_SMD:R_0603_1608Metric" V 1630 5900 50  0001 C CNN
 F 3 "~" H 1700 5900 50  0001 C CNN
@@
 AR Path="/60135668/6028372D" Ref="R534"  Part="1"
 F 0 "R534" H 1630 7009 50  0000 R CNN
-F 1 "8k2" H 1630 7100 50  0000 R CNN
+F 1 "82k" H 1630 7100 50  0000 R CNN
 F 2 "Resistor_SMD:R_0603_1608Metric" V 1630 7100 50  0001 C CNN
 F 3 "~" H 1700 7100 50  0001 C CNN
@@
 AR Path="/60135668/60283771" Ref="R530"  Part="1"
 F 0 "R530" H 3880 5809 50  0000 R CNN
-F 1 "1k" H 3880 5900 50  0000 R CNN
+F 1 "4k7" H 3880 5900 50  0000 R CNN
 F 2 "Resistor_SMD:R_0603_1608Metric" V 3880 5900 50  0001 C CNN
 F 3 "~" H 3950 5900 50  0001 C CNN
@@
 AR Path="/60135668/6028374A" Ref="R529"  Part="1"
 F 0 "R529" H 2980 5809 50  0000 R CNN
-F 1 "1k" H 2980 5900 50  0000 R CNN
+F 1 "10k" H 2980 5900 50  0000 R CNN
 F 2 "Resistor_SMD:R_0603_1608Metric" V 2980 5900 50  0001 C CNN
 F 3 "~" H 3050 5900 50  0001 C CNN
@@
 AR Path="/60135668/602C530E" Ref="R525"  Part="1"
 F 0 "R525" H 3080 4659 50  0000 R CNN
-F 1 "22k" H 3080 4750 50  0000 R CNN
+F 1 "10k" H 3080 4750 50  0000 R CNN
 F 2 "Resistor_SMD:R_0603_1608Metric" V 3080 4750 50  0001 C CNN
 F 3 "~" H 3150 4750 50  0001 C CNN
@@
 AR Path="/60135668/602CC487" Ref="R536"  Part="1"
 F 0 "R536" H 3080 7059 50  0000 R CNN
-F 1 "22k" H 3080 7150 50  0000 R CNN
+F 1 "10k" H 3080 7150 50  0000 R CNN
 F 2 "Resistor_SMD:R_0603_1608Metric" V 3080 7150 50  0001 C CNN
 F 3 "~" H 3150 7150 50  0001 C CNN
@@
 AR Path="/60135668/60328661" Ref="R520"  Part="1"
 F 0 "R520" H 7480 4359 50  0000 R CNN
-F 1 "470k" H 7480 4450 50  0000 R CNN
+F 1 "360k" H 7480 4450 50  0000 R CNN
 F 2 "Resistor_SMD:R_0603_1608Metric" V 7480 4450 50  0001 C CNN
 F 3 "~" H 7550 4450 50  0001 C CNN
@@
 AR Path="/60135668/60328668" Ref="R514"  Part="1"
 F 0 "R514" H 6880 3409 50  0000 R CNN
-F 1 "27k" H 6880 3500 50  0000 R CNN
+F 1 "20k" H 6880 3500 50  0000 R CNN
 F 2 "Resistor_SMD:R_0603_1608Metric" V 6880 3500 50  0001 C CNN
 F 3 "~" H 6950 3500 50  0001 C CNN
@@
 	6950 4450 6950 4550
 Text Notes 7300 3400 0    50   ~ 0
-17,5V +/-0,5V
+18,5V +/-0,5V
 $Comp
 L Device:R R?
@@
 AR Path="/60135668/6032868C" Ref="R515"  Part="1"
 F 0 "R515" H 8230 3409 50  0000 R CNN
-F 1 "1k" H 8230 3500 50  0000 R CNN
+F 1 "10k" H 8230 3500 50  0000 R CNN
 F 2 "Resistor_SMD:R_0603_1608Metric" V 8230 3500 50  0001 C CNN
 F 3 "~" H 8300 3500 50  0001 C CNN
@@
 AR Path="/60135668/603286B2" Ref="R516"  Part="1"
 F 0 "R516" H 9130 3409 50  0000 R CNN
-F 1 "1k" H 9130 3500 50  0000 R CNN
+F 1 "4k7" H 9130 3500 50  0000 R CNN
 F 2 "Resistor_SMD:R_0603_1608Metric" V 9130 3500 50  0001 C CNN
 F 3 "~" H 9200 3500 50  0001 C CNN
@@
 AR Path="/60135668/603286DB" Ref="R526"  Part="1"
 F 0 "R526" H 8330 4659 50  0000 R CNN
-F 1 "22k" H 8330 4750 50  0000 R CNN
+F 1 "10k" H 8330 4750 50  0000 R CNN
 F 2 "Resistor_SMD:R_0603_1608Metric" V 8330 4750 50  0001 C CNN
 F 3 "~" H 8400 4750 50  0001 C CNN

Commit message: Controller Rev2 fertig
Parts:
- R511: value 680k -> 270k
- R519: value 680k -> 470k
- R521: value 33k -> 22k
Changed lines of the file:
@@
 AR Path="/60135668/601CB1B5" Ref="R519"  Part="1"
 F 0 "R519" H 2280 4359 50  0000 R CNN
-F 1 "680k" H 2280 4450 50  0000 R CNN
+F 1 "470k" H 2280 4450 50  0000 R CNN
 F 2 "Resistor_SMD:R_0603_1608Metric" V 2280 4450 50  0001 C CNN
 F 3 "~" H 2350 4450 50  0001 C CNN
@@
 AR Path="/60135668/601CBE86" Ref="R511"  Part="1"
 F 0 "R511" H 1630 3409 50  0000 R CNN
-F 1 "680k" H 1630 3500 50  0000 R CNN
+F 1 "270k" H 1630 3500 50  0000 R CNN
 F 2 "Resistor_SMD:R_0603_1608Metric" V 1630 3500 50  0001 C CNN
 F 3 "~" H 1700 3500 50  0001 C CNN
@@
 AR Path="/60135668/601CC823" Ref="R521"  Part="1"
 F 0 "R521" H 1630 4609 50  0000 R CNN
-F 1 "33k" H 1630 4700 50  0000 R CNN
+F 1 "22k" H 1630 4700 50  0000 R CNN
 F 2 "Resistor_SMD:R_0603_1608Metric" V 1630 4700 50  0001 C CNN
 F 3 "~" H 1700 4700 50  0001 C CNN
