File: cad/pcb/saba-fernbedienung/rev2-a/6-audio.sch (KiCad schematic (older format))
At the start: 52 parts, among them U701 AD8656, U702 VS1053, Y701 12,288MHz

Commit message: ToDo-s bearbeitet
Parts:
- added C? (x2): 1u, Capacitor_SMD:C_0805_2012Metric, symbol Device:C
- added R? (x2): 220, Resistor_SMD:R_0603_1608Metric, symbol Device:R
- added T? (x2): Transformer_1P_1S, symbol Device:Transformer_1P_1S
- R706, R714: Placement (none) -> NP
- Y701: Bauteil ABM3-12.288MHZ-D2Y-T -> 12,2880-HC49-SMD
Connections:
- net Audio_Links: now also T?.4 (SB); no longer C705.1, R706.2
- net Audio_Rechts: now also T?.4 (SB); no longer C716.1, R714.2
- net GND: now also C?.1, C?.1, T?.2 (AB), T?.2 (AB); no longer R705.1, R713.1
- new net: C?.2, R705.1
- new net: C?.2, R713.1
- new net: R?.2, R?.2, T?.1 (AA)
- new net Audio_GND: T?.3 (SA), T?.3 (SA)
- new net amp_links: C705.1, R706.2, R?.1
- new net amp_rechts: C716.1, R714.2, R?.1, T?.1 (AA)
Other:
- note added: "Massetrennung\n"
- note added: "Optional: Stereo - 2x 0R,\n2x Übertrager"
- note added: "Power"
- moved on the sheet: C716, C718, R706, R708, R709, R710, R712, R713, R714, RV702, U701B

Commit message: Change: Bauteilbezeichner
Parts:
- gave numbers to parts that had none: 6
- renumbered C714 to C715, C715 to C716, C716 to C718, C718 to C720, C720 to C722, C721 to C723, C722 to C724, C723 to C725, C724 to C726, C725 to C727, R711 to R710, R710 to R711, R715 to R712, R712 to R713, R713 to R714, R716 to R715, R717 to R716, R718 to R717, R714 to R718

Commit message: Sicherung
Parts:
- T701, T702: value Transformer_1P_1S -> 1:1; footprint (none) -> local:Transformer_NF_EI14
Other:
- note added: "Optional: Stereo - 1x 0R,\n2x Übertrager"
- note removed: "Optional: Stereo - 2x 0R,\n2x Übertrager"
Changed lines of the file:
@@
 P 5100 6400
 F 0 "T701" H 5100 6781 50  0000 C CNN
-F 1 "Transformer_1P_1S" H 5100 6690 50  0000 C CNN
-F 2 "" H 5100 6400 50  0001 C CNN
+F 1 "1:1" H 5100 6690 50  0000 C CNN
+F 2 "local:Transformer_NF_EI14" H 5100 6400 50  0001 C CNN
 F 3 "~" H 5100 6400 50  0001 C CNN
 	1    5100 6400
@@
 P 5100 7100
 F 0 "T702" H 5100 7500 50  0000 C CNN
-F 1 "Transformer_1P_1S" H 5100 7400 50  0000 C CNN
-F 2 "" H 5100 7100 50  0001 C CNN
+F 1 "1:1" H 5100 7400 50  0000 C CNN
+F 2 "local:Transformer_NF_EI14" H 5100 7100 50  0001 C CNN
 F 3 "~" H 5100 7100 50  0001 C CNN
 F 4 "NP" H 5100 6800 50  0000 C CNN "Placement"
@@
 amp_rechts
 Text Notes 3250 7150 0    50   ~ 0
-Optional: Stereo - 2x 0R,\n2x Übertrager
+Optional: Stereo - 1x 0R,\n2x Übertrager
 Text GLabel 5650 7300 2    50   Output ~ 0
 Audio_GND
